File: Hardware/hw/_autosave-hw.kicad_pcb (KiCad board)
At the start: 2 copper layers, 2 parts, among them U1 ESP32-C6-WROOM-1, U2 RV-3028-C7

Commit message: Scheme update
Parts:
- added C1: C, Capacitor_SMD:C_0805_2012Metric, F.Cu at (136.7, 68.5)
- added J1: Screw_Terminal_01x02, TerminalBlock:TerminalBlock_Xinya_XY308-2.54-2P_1x02_P2.54mm_Horizontal, F.Cu at (149.0, 59.0)
- added J1: Screw_Terminal_01x02, TerminalBlock_Phoenix:TerminalBlock_Phoenix_MPT-0,5-2-2.54_1x02_P2.54mm_Horizontal, F.Cu at (151.5, 83.5)
- added Q1: FS8205A, FS8205A:SOP65P640X120-8N, F.Cu at (152.6, 101.5)
- added R1: R, Resistor_SMD:R_0805_2012Metric, F.Cu at (141.1, 68.5)
- added U3: INA219, INA219:MODULE_INA219, F.Cu at (78.0, 89.0)
- added U4: SC189LSKTRT, SC189LSKTRT:SOT95P280X145-5N, F.Cu at (120.0, 112.5)
- added U5: TP4056-42-ESOP8, Package_SO:SOIC-8-1EP_3.9x4.9mm_P1.27mm_EP2.41x3.3mm_ThermalVias, F.Cu at (119.8, 104.0)
- added U6: TPS63002DRCT, TPS63002DRCT:VREG_V62_16624-01YE, F.Cu at (142.1, 107.0)
Connections:
- net Net-(U1-GND-Pad1) renamed GND
- U1 pad 6: unconnected-(U1-MTCK/GPIO6/ADC1_CH6-Pad6) -> I2C_SDA
- U1 pad 7: unconnected-(U1-MTDO/GPIO7-Pad7) -> I2C_SCL
- U2 pad 3: unconnected-(U2-SCL-Pad3) -> I2C_SCL
- U2 pad 4: unconnected-(U2-SDA-Pad4) -> I2C_SDA
