File: Hardware/hw/_autosave-hw.kicad_pcb (KiCad board)
At the start: 2 copper layers, 21 parts, among them J1 Screw_Terminal_01x02, J2 Screw_Terminal_01x02, J3 Conn_01x05_Pin, J5 Conn_01x04_Pin, Q1 FS8205A, U1 ESP32-C6-WROOM-1, U2 RV-3028-C7, U4 SC189LSKTRT, U5 TP4056-42-ESOP8, U6 TPS63002DRCT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

Commit message: update
Parts:
- D3: footprint MyESDProtection:SMS3.3.TCT -> SMBJ24CA:DO214AA
Changed lines of the file:
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@@
 	(net 72 "SCL")
 	(net 73 "Charging")
-	(footprint "MyESDProtection:SMS3.3.TCT"
+	(footprint "SMBJ24CA:DO214AA"
 		(layer "F.Cu")
 		(at 121.4 75.55)
-		(descr "6-pin SOT-23 package")
-		(tags "SOT-23-6")
+		(descr "Diode SMB Standard")
+		(tags "Diode SMB Standard")
 		(property "Reference" "D3"
-			(at 0 -2.9 0)
-			(layer "F.SilkS")
+			(at 0.5 0 0)
+			(layer "F.Fab")
 			(effects
 				(font
@@
 		)
 		(property "Value" "~"
-			(at 0 2.9 0)
-			(layer "F.Fab")
+			(at 0.05 4.7 0)
+			(layer "F.Fab")
+			(hide yes)
 			(effects
 				(font
@@
 		(attr smd)
 		(fp_line
-			(start -0.9 1.61)
-			(end 0.9 1.61)
-			(stroke
-				(width 0.12)
+			(start -2.30632 1.8)
+			(end -2.30632 1.6002)
+			(stroke
+				(width 0.15)
+				(type solid)
+			)
+			(layer "F.SilkS")
+		)
+		(fp_line
+			(start -2.30632 1.99644)
+			(end -2.30632 1.79832)
+			(stroke
+				(width 0.15)
+				(type solid)
+			)
+			(layer "F.SilkS")
+		)
+		(fp_line
+			(start -2.30632 1.99644)
+			(end 2.29616 1.99644)
+			(stroke
+				(width 0.15)
+				(type solid)
+			)
+			(layer "F.SilkS")
+		)
+		(fp_line
+			(start -2.30124 -1.99898)
+			(end -2.30124 -1.80086)
+			(stroke
+				(width 0.15)
+				(type solid)
+			)
+			(layer "F.SilkS")
+		)
+		(fp_line
+			(start -2.30124 -1.99898)
+			(end 2.30124 -1.99898)
+			(stroke
+				(width 0.15)
+				(type solid)
+			)
+			(layer "F.SilkS")
+		)
+		(fp_line
+			(start -2.30124 -1.8)
+			(end -2.30124 -1.651)
+			(stroke
+				(width 0.15)
+				(type solid)
+			)
+			(layer "F.SilkS")
+		)
+		(fp_line
+			(start -1.84928 -1.99898)
+			(end -1.84928 -1.80086)
+			(stroke
+				(width 0.15)
+				(type solid)
+			)
+			(layer "F.SilkS")
+		)
+		(fp_line
+			(start -1.84928 -1.8)
+			(end -1.84928 -1.651)
+			(stroke
+				(width 0.15)
+				(type solid)
+			)
+			(layer "F.SilkS")
+		)
+		(fp_line
+			(start -1.84928 1.75)
+			(end -1.84928 1.601)
+			(stroke
+				(width 0.15)
+				(type solid)
+			)
+			(layer "F.SilkS")
+		)
+		(fp_line
+			(start -1.84928 1.94898)
+			(end -1.84928 1.75086)
+			(stroke
+				(width 0.15)
+				(type solid)
+			)
+			(layer "F.SilkS")
+		)
+		(fp_line
+			(start 2.29616 1.8)
+			(end 2.29616 1.651)
+			(stroke
+				(width 0.15)
+				(type solid)
+			)
+			(layer "F.SilkS")
+		)
+		(fp_line
+			(start 2.29616 1.99644)
+			(end 2.29616 1.79832)
+			(stroke
+				(width 0.15)
+				(type solid)
+			)
+			(layer "F.SilkS")
+		)
+		(fp_line
+			(start 2.30124 -1.99898)
+			(end 2.30124 -1.80086)
+			(stroke
+				(width 0.15)
+				(type solid)
+			)
+			(layer "F.SilkS")
+		)
+		(fp_line
+			(start 2.30124 -1.8)
+			(end 2.30124 -1.651)
+			(stroke
+				(width 0.15)
 				(type solid)
 			)
@@
 		)
 		(fp_circle
-			(center -1.297926 -1.5)
-			(end -1.195518 -1.5)
-			(stroke
-				(width 0.1)
-				(type solid)
-			)
-			(fill yes)
-			(layer "F.SilkS")
-		)
-		(fp_line
-			(start -1.9 -1.8)
-			(end -1.9 1.8)
-			(stroke
-				(width 0.05)
-				(type solid)
-			)
-			(layer "F.CrtYd")
-		)
-		(fp_line
-			(start -1.9 1.8)
-			(end 1.9 1.8)
-			(stroke
-				(width 0.05)
-				(type solid)
-			)
-			(layer "F.CrtYd")
-		)
-		(fp_line
-			(start 1.9 -1.8)
-			(end -1.9 -1.8)
-			(stroke
-				(width 0.05)
-				(type solid)
-			)
-			(layer "F.CrtYd")
-		)
-		(fp_line
-			(start 1.9 1.8)
-			(end 1.9 -1.8)
-			(stroke
-				(width 0.05)
-				(type solid)
-			)
-			(layer "F.CrtYd")
-		)
-		(fp_line
-			(start -0.9 -1.55)
-			(end -0.9 -0.5)
-			(stroke
-				(width 0.1)
-				(type solid)
-			)
-			(layer "F.Fab")
-		)
-		(fp_line
-			(start -0.9 -0.9)
-			(end -0.9 1.55)
-			(stroke
-				(width 0.1)
-				(type solid)
-			)
-			(layer "F.Fab")
-		)
-		(fp_line
-			(start 0.9 -1.55)
-			(end -0.9 -1.55)
-			(stroke
-				(width 0.1)
-				(type solid)
-			)
-			(layer "F.Fab")
-		)
-		(fp_line
-			(start 0.9 -1.55)
-			(end 0.9 1.55)
-			(stroke
-				(width 0.1)
-				(type solid)
-			)
-			(layer "F.Fab")
-		)
-		(fp_line
-			(start 0.9 1.55)
-			(end -0.9 1.55)
-			(stroke
-				(width 0.1)
+			(center 0 0)
+			(end 0.20066 0.09906)
+			(stroke
+				(width 0.381)
+				(type solid)
+			)
+			(fill no)
+			(layer "F.Adhes")
+		)
+		(fp_circle
+			(center 0 0)
+			(end 0.44958 0.09906)
+			(stroke
+				(width 0.381)
+				(type solid)
+			)
+			(fill no)
+			(layer "F.Adhes")
+		)
+		(fp_line
+			(start -3.75 -2.25)
+			(end -3.75 2.25)
+			(stroke
+				(width 0.0508)
+				(type solid)
+			)
+			(layer "F.Fab")
+		)
+		(fp_line
+			(start -3.75 2.25)
+			(end 3.75 2.25)
+			(stroke
+				(width 0.0508)
+				(type solid)
+			)
+			(layer "F.Fab")
+		)
+		(fp_line
+			(start -2.794 -2.2352)
+			(end -2.794 2.2606)
+			(stroke
+				(width 0.0508)
+				(type solid)
+			)
+			(layer "F.Fab")
+		)
+		(fp_line
+			(start 3.75 -2.25)
+			(end -3.75 -2.25)
+			(stroke
+				(width 0.0508)
+				(type solid)
+			)
+			(layer "F.Fab")
+		)
+		(fp_line
+			(start 3.75 2.25)
+			(end 3.75 -2.25)
+			(stroke
+				(width 0.0508)
 				(type solid)
 			)
@@
 		)
 		(fp_text user "${REFERENCE}"
-			(at 0 0 0)
-			(layer "F.Fab")
-			(effects
-				(font
-					(size 0.5 0.5)
-					(thickness 0.075)
-				)
-			)
-		)
-		(pad "1" smd roundrect
-			(at -1.1 -0.95)
-			(size 1.1 0.65)
+			(at -4.75 0 90)
+			(layer "F.SilkS")
+			(effects
+				(font
+					(size 1 1)
+					(thickness 0.15)
+				)
+			)
+		)
+		(pad "1" smd rect
+			(at -2.14884 0)
+			(size 2.49936 2.30124)
 			(layers "F.Cu" "F.Mask" "F.Paste")
-			(roundrect_rratio 0.2)
 			(net 17 "Net-(J1-Pin_2)")
 			(pintype "passive")
 		)
-		(pad "2" smd roundrect
-			(at -1.1 0)
-			(size 1.1 0.65)
+		(pad "2" smd rect
+			(at 2.14884 0)
+			(size 2.49936 2.30124)
 			(layers "F.Cu" "F.Mask" "F.Paste")
-			(roundrect_rratio 0.2)
 			(net 38 "GND")
 			(pintype "passive")
 		)
-		(pad "3" smd roundrect
-			(at -1.1 0.95)
-			(size 1.1 0.65)
-			(layers "F.Cu" "F.Mask" "F.Paste")
-			(roundrect_rratio 0.2)
-		)
-		(pad "4" smd roundrect
-			(at 1.1 0.95)
-			(size 1.1 0.65)
-			(layers "F.Cu" "F.Mask" "F.Paste")
-			(roundrect_rratio 0.2)
-		)
-		(pad "5" smd roundrect
-			(at 1.1 0)
-			(size 1.1 0.65)
-			(layers "F.Cu" "F.Mask" "F.Paste")
-			(roundrect_rratio 0.2)
-		)
-		(pad "6" smd roundrect
-			(at 1.1 -0.95)
-			(size 1.1 0.65)
-			(layers "F.Cu" "F.Mask" "F.Paste")
-			(roundrect_rratio 0.2)
-		)
 		(embedded_fonts no)
-		(model "${KICAD8_3DMODEL_DIR}/Package_TO_SOT_SMD.3dshapes/SOT-23-6.step"
-			(offset
-				(xyz 0 0 0)
-			)
-			(scale
-				(xyz 1 1 1)
-			)
-			(rotate
-				(xyz 0 0 0)
-			)
-		)
 	)
 	(footprint "Connector_PinSocket_2.54mm:PinSocket_1x05_P2.54mm_Vertical"
