File: Hardware/hw/_autosave-hw.kicad_pcb (KiCad board)
At the start: 2 copper layers, 130.6 x 81.9 mm, 113 parts, among them J1 Screw_Terminal_01x02, J10 Screw_Terminal_01x02, J2 Screw_Terminal_01x03, J3 Conn_01x04_Pin, J4 USB4085-GF-A_REVA4, J5 Screw_Terminal_01x04, J6 Screw_Terminal_01x04, J7 Screw_Terminal_01x04, J8 Screw_Terminal_01x04, J9 Screw_Terminal_01x04, Q1 PMOS, Q10 NMOS, Q11 NMOS, Q12 NMOS, Q13 NMOS, Q14 NMOS, Q15 NMOS, Q16 NMOS, Q17 NMOS, Q18 NMOS, Q19 NMOS, Q2 PMOS, Q3 NMOS, Q4 PMOS, Q5 PMOS, Q6 PMOS, Q7 PMOS, Q8 NMOS, Q9 NMOS, SW1 SW_Push, SW2 SW_Push, U1 INA219, U10 PESD5V0L2BT,215, U11 PESD5V0L2BT,215, U12 PESD5V0L2BT,215, U13 MCP3422A0-E/SN, U2 INA219, U3 SunnyBuddy:PRT-12885, U4 ESP32-C6-WROOM-1, U5 TPS63001, U6 USBLC6-4SC6, U7 RV-3028-C7, U8 PESD5V0L2BT,215, U9 PESD5V0L2BT,215

Commit message: PCB update
Routing:
- net I2C_SCL: track 108.6 -> 261.0 mm, vias 0 -> 9
- net I2C_SDA: track 143.7 -> 269.4 mm, vias 0 -> 10
- net +3V3: track 360.6 -> 456.6 mm, vias 3 -> 12
- net Data-: track 8.49 -> 79.4 mm, vias 0 -> 1
- net GPIO20: track 0.00 -> 65.4 mm, vias 0 -> 2
- net GPIO10: track 0.00 -> 64.5 mm, vias 0 -> 4
- net RST: track 7.59 -> 51.6 mm, vias 0 -> 2
- net GPIO15: track 0.00 -> 38.3 mm, vias 0 -> 2
- net GPIO11: track 0.00 -> 37.5 mm, vias 0 -> 4
- net Net-(U7-VBACKUP): track 0.00 -> 25.4 mm, vias 0 -> 6
- net GPIO0: track 15.0 -> 36.1 mm, vias 0 -> 4
- net GPIO18: track 0.00 -> 17.5 mm, vias 0 -> 2
- net Data+: track 63.9 -> 65.8 mm
- net BOOT: track 67.6 -> 69.2 mm, vias 0 -> 2
- net Net-(U7-EVI): track 11.1 -> 12.6 mm
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