File: Hardware/hw/_autosave-charging.kicad_sch (KiCad schematic)
At the start: 11 parts, among them J1 Screw_Terminal_01x02, J2 Screw_Terminal_01x02, Q2 PMOS, Q3 PMOS, Q4 PMOS, U3 INA219, U7 BQ24650, U8 PRT-12885

Commit message: update
Parts:
- removed U3: INA219, INA219:MODULE_INA219, symbol INA219:INA219
- removed U7: BQ24650, symbol BQ24650:BQ24650
- removed U8: PRT-12885, symbol PRT-12885:Sunny Buddy PRT-12885
- added J3: Conn_01x05_Pin, Connector_PinSocket_2.54mm:PinSocket_1x05_P2.54mm_Vertical, symbol Connector:Conn_01x05_Pin
- added J5: Conn_01x04_Pin, Connector_PinSocket_2.54mm:PinSocket_1x04_P2.54mm_Vertical, symbol Connector:Conn_01x04_Pin
- added R5, R6: 4k7, symbol Device:R
- added R7, R8: 10k, symbol Device:R
- added SunnyBuddy:PRT-12885: ~, SunnyBuddy:PRT-12885, symbol PRT-12885:Sunny Buddy PRT-12885
- added U7: INA219, INA219_Module:MODULE_INA219, symbol INA219:INA219
- D3: footprint (none) -> SMBJ24CA:DO214AA
Connections:
- net GND: now also J3.5 (Pin_5), J5.4 (Pin_4), SunnyBuddy:PRT-12885.2 (Sol-), SunnyBuddy:PRT-12885.4 (GND), U7.2 (GND)
- net Charging: now reaches R4.2
- net Charging: now also J3.4 (Pin_4)
- net at J2.1 (Pin_1): now also SunnyBuddy:PRT-12885.7 (LOAD+)
- net at J2.2 (Pin_2): now also SunnyBuddy:PRT-12885.8 (LOAD-)
- net at Q4.1 (D): now also U7.6 (VIN+)
- new net: SunnyBuddy:PRT-12885.1 (Sol+), U7.5 (VIN-)
- new net CHG: J5.3 (Pin_3), R8.2, SunnyBuddy:PRT-12885.6 (CHG)
- new net FAULT: J5.2 (Pin_2), R7.2, SunnyBuddy:PRT-12885.5 (FAULT)
- new net SCL: J3.2 (Pin_2), R5.2, U7.3 (SCL)
- new net SDA: J3.3 (Pin_3), R6.2, U7.4 (SDA)
- new net SET: J5.1 (Pin_1), SunnyBuddy:PRT-12885.3 (SET)
- new net VCC: J3.1 (Pin_1), R5.1, R6.1, R7.1, R8.1, U7.1 (VCC)
Other:
- moved on the sheet: J2
