File: Hardware/hw/hw.kicad_sch (KiCad schematic)
At the start: 2 parts, among them U1 ESP32-C6-WROOM-1, U2 RV-3028-C7

Commit message: Scheme update
Parts:
- added C1: C, Capacitor_SMD:C_0805_2012Metric, symbol Device:C
- added C2: 0,1uF, Capacitor_SMD:C_0805_2012Metric, symbol Device:C
- added C3, C4, C5: 10uF, Capacitor_SMD:C_0805_2012Metric, symbol Device:C
- added J1, J2: Screw_Terminal_01x02, TerminalBlock_Phoenix:TerminalBlock_Phoenix_MPT-0,5-2-2.54_1x02_P2.54mm_Horizontal, symbol Connector:Screw_Terminal_01x02
- added L1: 2.2uH, Inductor_SMD:L_0201_0603Metric, symbol Device:L
- added Q1: FS8205A, FS8205A:SOP65P640X120-8N, symbol FS8205A:FS8205A
- added R1: R, Resistor_SMD:R_0805_2012Metric, symbol Device:R
- added R2: 100R, Resistor_SMD:R_0805_2012Metric, symbol Device:R
- added U3: INA219, INA219:MODULE_INA219, symbol INA219:INA219
- added U4: SC189LSKTRT, SC189LSKTRT:SOT95P280X145-5N, symbol SC189LSKTRT:SC189LSKTRT
- added U5: TP4056-42-ESOP8, Package_SO:SOIC-8-1EP_3.9x4.9mm_P1.27mm_EP2.41x3.3mm_ThermalVias, symbol Battery_Management:TP4056-42-ESOP8
- added U6: TPS63002DRCT, TPS63002DRCT:VREG_V62_16624-01YE, symbol TPS63002DRCT:TPS63002DRCT
Connections:
- net I2C_SCL: now reaches U2.3 (SCL)
- net I2C_SCL: now also U1.7 (MTDO/GPIO7)
- net I2C_SDA: now reaches U2.4 (SDA)
- net I2C_SDA: now also U1.6 (MTCK/GPIO6/ADC1_CH6)
- net GND: now reaches U1.1 (GND), U1.28 (GND), U1.29 (GND)
- net GND: now also C2.2, C3.2, C4.2, C5.2, J1.1 (Pin_1), U6.11 (POWER_PAD), U6.3 (PGND), U6.9 (GND)
- new net: L1.1, U6.4 (L1)
- new net: L1.2, U6.2 (L2)
- new net: C2.1, R2.2, U6.6 (EN), U6.7 (PS/SYNC), U6.8 (VINA)
- new net: J1.2 (Pin_2), U3.6 (VIN+), U3.VIN+
- new net: C3.1, R2.1, U3.1 (VCC), U6.5 (VIN)
- new net: U3.5 (VIN-), U3.VIN-
- new net: U3.SH1 (SHIELD), U3.SH2 (SHIELD), U3.SH3 (SHIELD), U3.SH4 (SHIELD)
- new net: Q1.1, Q1.8
- new net: Q1.2, Q1.3
- new net: Q1.6, Q1.7
- new net FB-VOUT: C4.1, C5.1, U5.4 (V_{CC}), U6.1 (VOUT), U6.10 (FB)
Other:
- added sheet blokovka (blokovka.kicad_sch)
- moved on the sheet: U1, U2

Commit message: lib update
Parts:
- added U7: ~, symbol BQ24650:BQ24650
Other:
- moved on the sheet: U2
Changed lines of the file:
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@@
+		)
+	)
+	(wire
+		(pts
+			(xy 31.75 124.46) (xy 26.67 124.46)
+		)
+		(stroke
+			(width 0)
+			(type default)
+		)
+	)
+	(wire
+		(pts
+			(xy 31.75 121.92) (xy 26.67 121.92)
+		)
+		(stroke
+			(width 0)
+			(type default)
 		)
 	)
@@
 	(symbol
 		(lib_id "Timer_RTC:RV-3028-C7")
-		(at 39.37 127 0)
+		(at 44.45 127 0)
 		(unit 1)
 		(exclude_from_sim no)
@@
 		(fields_autoplaced yes)
 		(property "Reference" "U2"
-			(at 41.5133 137.16 0)
+			(at 46.5933 137.16 0)
 			(effects
 				(font
@@
 		)
 		(property "Value" "RV-3028-C7"
-			(at 41.5133 139.7 0)
+			(at 46.5933 139.7 0)
 			(effects
 				(font
@@
 		)
 		(property "Footprint" "Package_SON:MicroCrystal_C7_SON-8_1.5x3.2mm_P0.9mm"
-			(at 64.77 135.89 0)
+			(at 69.85 135.89 0)
 			(effects
 				(font
@@
 		)
 		(property "Datasheet" "https://www.microcrystal.com/fileadmin/Media/Products/RTC/Datasheet/RV-3028-C7.pdf"
-			(at 39.37 127 0)
+			(at 44.45 127 0)
 			(effects
 				(font
@@
 		)
 		(property "Description" "Realtime Clock/Calendar I2C Interface, Extreme Low Power, 1.1 V to 5.5 V, MicroCrystal C7"
-			(at 39.37 127 0)
+			(at 44.45 127 0)
 			(effects
 				(font
@@
 					(unit 1)
 				)
+			)
+		)
+	)
+	(symbol
+		(lib_id "BQ24650:BQ24650")
+		(at 88.9 96.52 0)
+		(unit 1)
+		(exclude_from_sim no)
+		(in_bom yes)
+		(on_board yes)
+		(dnp no)
+		(fields_autoplaced yes)
+		(property "Reference" "U7"
+			(at 88.265 92.71 0)
+			(effects
+				(font
+					(size 1.27 1.27)
+				)
+			)
+		)
+		(property "Value" "~"
+			(at 88.265 95.25 0)
+			(effects
+				(font
+					(size 1.27 1.27)
+				)
+			)
+		)
+		(property "Footprint" ""
+			(at 88.9 96.52 0)
+			(effects
+				(font
+					(size 1.27 1.27)
+				)
+				(hide yes)
+			)
+		)
+		(property "Datasheet" ""
+			(at 88.9 96.52 0)
+			(effects
+				(font
+					(size 1.27 1.27)
+				)
+				(hide yes)
+			)
+		)
+		(property "Description" ""
+			(at 88.9 96.52 0)
+			(effects
+				(font
+					(size 1.27 1.27)
+				)
+				(hide yes)
+			)
+		)
+		(pin "4"
+		)
+		(pin "3"
+		)
+		(pin "2"
+		)
+		(pin "1"
+		)
+		(instances
+			(project ""
+				(path "/e8888c0f-4960-4960-b96f-1ca6e03d7c29"
+					(reference "U7")
+					(unit 1)
+				)

Commit message: Charging update
Parts:
- removed J1, J2: Screw_Terminal_01x02, TerminalBlock_Phoenix:TerminalBlock_Phoenix_MPT-0,5-2-2.54_1x02_P2.54mm_Horizontal, symbol Connector:Screw_Terminal_01x02
- removed U3: INA219, INA219:MODULE_INA219, symbol INA219:INA219
- removed U7: ~, symbol BQ24650:BQ24650
Other:
- added sheet Charging logic (charging.kicad_sch)
- moved on the sheet: C2, C3, C4, C5, L1, R2, U5, U6

Commit message: IoT board update
Parts:
- removed C2: 0,1uF, Capacitor_SMD:C_0805_2012Metric, symbol Device:C
- removed C3, C4, C5: 10uF, Capacitor_SMD:C_0805_2012Metric, symbol Device:C
- removed L1: 2.2uH, Inductor_SMD:L_0201_0603Metric, symbol Device:L
- removed R2: 100R, Resistor_SMD:R_0805_2012Metric, symbol Device:R
- removed U1: ESP32-C6-WROOM-1, PCM_Espressif:ESP32-C6-WROOM-1, symbol PCM_Espressif:ESP32-C6-WROOM-1
- removed U2: RV-3028-C7, Package_SON:MicroCrystal_C7_SON-8_1.5x3.2mm_P0.9mm, symbol Timer_RTC:RV-3028-C7
- removed U5: TP4056-42-ESOP8, Package_SO:SOIC-8-1EP_3.9x4.9mm_P1.27mm_EP2.41x3.3mm_ThermalVias, symbol Battery_Management:TP4056-42-ESOP8
- removed U6: TPS63002DRCT, TPS63002DRCT:VREG_V62_16624-01YE, symbol TPS63002DRCT:TPS63002DRCT
Other:
- added sheet IoTdevice (iot_device.kicad_sch)
- sheet Charging logic ports: added green; removed none

Commit message: IoT update
Parts:
- removed C1: C, Capacitor_SMD:C_0805_2012Metric, symbol Device:C
- removed Q1: FS8205A, FS8205A:SOP65P640X120-8N, symbol FS8205A:FS8205A
- removed R1: R, Resistor_SMD:R_0805_2012Metric, symbol Device:R
- removed U4: SC189LSKTRT, SC189LSKTRT:SOT95P280X145-5N, symbol SC189LSKTRT:SC189LSKTRT
Other:
- added sheet garbage (garbage.kicad_sch)

Commit message: Big update
Other:
- sheet Charging logic renamed Charging
- sheet IoTdevice renamed ESP32
- removed sheet blokovka
- added sheet Sensors (sensors.kicad_sch)
Changed lines of the file:
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@@
 			(color 0 0 0 0.0000)
 		)
-		(property "Sheetname" "IoTdevice"
+		(property "Sheetname" "ESP32"
 			(at 44.45 65.3284 0)
 			(effects
@@
 			(project "hw"
 				(path "/e8888c0f-4960-4960-b96f-1ca6e03d7c29"
-					(page "4")
-				)
-			)
-		)
-	)
-	(sheet
-		(at 95.25 19.05)
-		(size 12.7 3.81)
-		(exclude_from_sim no)
-		(in_bom yes)
-		(on_board yes)
-		(dnp no)
-		(fields_autoplaced yes)
-		(stroke
-			(width 0.1524)
-			(type solid)
-		)
-		(fill
-			(color 0 0 0 0.0000)
-		)
-		(property "Sheetname" "blokovka"
-			(at 95.25 18.3384 0)
-			(effects
-				(font
-					(size 1.27 1.27)
-				)
-				(justify left bottom)
-			)
-		)
-		(property "Sheetfile" "blokovka.kicad_sch"
-			(at 95.25 23.4446 0)
-			(effects
-				(font
-					(size 1.27 1.27)
-				)
-				(justify left top)
-			)
-		)
-		(property "Field2" ""
-			(at 95.25 19.05 0)
-			(effects
-				(font
-					(size 1.27 1.27)
-				)
-			)
-		)
-		(instances
-			(project "hw"
-				(path "/e8888c0f-4960-4960-b96f-1ca6e03d7c29"
-					(page "2")
+					(page "3")
 				)
 			)
@@
 			(color 0 0 0 0.0000)
 		)
-		(property "Sheetname" "Charging logic"
+		(property "Sheetname" "Charging"
 			(at 44.45 17.0684 0)
 			(effects
@@
 			(project "hw"
 				(path "/e8888c0f-4960-4960-b96f-1ca6e03d7c29"
-					(page "3")
+					(page "2")
 				)
 			)
+		)
+	)
+	(sheet
+		(at 104.14 121.92)
+		(size 24.13 17.78)
+		(exclude_from_sim no)
+		(in_bom yes)
+		(on_board yes)
+		(dnp no)
+		(fields_autoplaced yes)
+		(stroke
+			(width 0.1524)
+			(type solid)
+		)
+		(fill
+			(color 0 0 0 0.0000)
+		)
+		(property "Sheetname" "Sensors"
+			(at 104.14 121.2084 0)
+			(effects
+				(font
+					(size 1.27 1.27)
+				)
+				(justify left bottom)
+			)
+		)
+		(property "Sheetfile" "sensors.kicad_sch"
+			(at 104.14 140.2846 0)
+			(effects
+				(font
+					(size 1.27 1.27)
+				)
+				(justify left top)
+			)
+		)
+		(instances
+			(project "hw"
+				(path "/e8888c0f-4960-4960-b96f-1ca6e03d7c29"
+					(page "4")
+				)
+			)

Commit message: little update
Other:
- removed sheet garbage
Changed lines of the file:
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@@
-	)
-	(sheet
-		(at 143.51 67.31)
-		(size 22.86 15.24)
-		(exclude_from_sim no)
-		(in_bom yes)
-		(on_board yes)
-		(dnp no)
-		(fields_autoplaced yes)
-		(stroke
-			(width 0.1524)
-			(type solid)
-		)
-		(fill
-			(color 0 0 0 0.0000)
-		)
-		(property "Sheetname" "garbage"
-			(at 143.51 66.5984 0)
-			(effects
-				(font
-					(size 1.27 1.27)
-				)
-				(justify left bottom)
-			)
-		)
-		(property "Sheetfile" "garbage.kicad_sch"
-			(at 143.51 83.1346 0)
-			(effects
-				(font
-					(size 1.27 1.27)
-				)
-				(justify left top)
-			)
-		)
-		(instances
-			(project "hw"
-				(path "/e8888c0f-4960-4960-b96f-1ca6e03d7c29"
-					(page "5")
-				)
-			)
-		)
 	)
 	(sheet
@@
 	)
 	(sheet
-		(at 104.14 121.92)
+		(at 110.49 43.18)
 		(size 24.13 17.78)
 		(exclude_from_sim no)
@@
 		)
 		(property "Sheetname" "Sensors"
-			(at 104.14 121.2084 0)
+			(at 110.49 42.4684 0)
 			(effects
 				(font
@@
 		)
 		(property "Sheetfile" "sensors.kicad_sch"
-			(at 104.14 140.2846 0)
+			(at 110.49 61.5446 0)
 			(effects
 				(font

Commit message: Hardware v1.0
Other:
- sheet Charging ports: added none; removed green
- company: (none) -> UNIZA Faculty of Management Science and Informatics Department of Technical Cybernetics
- title: (none) -> Solar Power Management and Monitoring Circuit
Changed lines of the file:
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@@
 	(generator_version "9.0")
 	(paper "A4")
+	(title_block
+		(title "Solar Power Management and Monitoring Circuit")
+		(date "2026-04-24")
+		(rev "Tomáš Bača")
+		(company "UNIZA Faculty of Management Science and Informatics Department of Technical Cybernetics")
+		(comment 1 "Author: Peter Kolok")
+	)
 	(sheet
-		(at 44.45 66.04)
-		(size 31.75 16.51)
+		(at 104.14 17.78)
+		(size 48.26 40.64)
 		(exclude_from_sim no)
 		(in_bom yes)
@@
 		)
 		(property "Sheetname" "ESP32"
-			(at 44.45 65.3284 0)
+			(at 104.14 17.0684 0)
 			(effects
 				(font
@@
 		)
 		(property "Sheetfile" "iot_device.kicad_sch"
-			(at 44.45 83.1346 0)
+			(at 104.14 59.0046 0)
 			(effects
 				(font
@@
 	(sheet
 		(at 44.45 17.78)
-		(size 26.67 16.51)
+		(size 48.26 41.91)
 		(exclude_from_sim no)
 		(in_bom yes)
@@
 		)
 		(property "Sheetfile" "charging.kicad_sch"
-			(at 44.45 34.8746 0)
+			(at 44.45 60.2746 0)
 			(effects
 				(font
@@
 				)
 				(justify left top)
-			)
-		)
-		(pin "green" input
-			(at 71.12 22.86 0)
-			(effects
-				(font
-					(size 1.27 1.27)
-				)
-				(justify right)
 			)
 		)
@@
 	)
 	(sheet
-		(at 110.49 43.18)
-		(size 24.13 17.78)
+		(at 163.83 17.78)
+		(size 49.53 40.64)
 		(exclude_from_sim no)
 		(in_bom yes)
@@
 		)
 		(property "Sheetname" "Sensors"
-			(at 110.49 42.4684 0)
+			(at 163.83 17.0684 0)
 			(effects
 				(font
@@
 		)
 		(property "Sheetfile" "sensors.kicad_sch"
-			(at 110.49 61.5446 0)
+			(at 163.83 59.0046 0)
 			(effects
 				(font
