File: Hardware/hw/hw.kicad_pcb (KiCad board)
At the start: 2 copper layers, 21 parts, among them J1 Screw_Terminal_01x02, J2 Screw_Terminal_01x02, J3 Conn_01x05_Pin, J5 Conn_01x04_Pin, Q1 FS8205A, U1 ESP32-C6-WROOM-1, U2 RV-3028-C7, U4 SC189LSKTRT, U5 TP4056-42-ESOP8, U6 TPS63002DRCT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

Commit message: SMS3.3.TCT update
Parts:
- moved U1 95.8 mm to (160.0, 85.5)
Changed lines of the file:
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@@
 	(footprint "PCM_Espressif:ESP32-C6-WROOM-1"
 		(layer "F.Cu")
-		(at 67.365 109.915)
+		(at 160 85.5)
 		(descr "ESP32-C6-WROOM-1: https://www.espressif.com/sites/default/files/documentation/esp32-c6-wroom-1_datasheet_en.pdf")
 		(tags "esp32-c6")
@@
 			(polygon
 				(pts
-					(xy 76.365 100.165) (xy 58.365 100.165) (xy 58.365 94.165) (xy 76.365 94.165)
-				)
-			)
+					(xy 169 75.75) (xy 151 75.75) (xy 151 69.75) (xy 169 69.75)
+				)
+			)

Commit message: scheme update
Parts:
- added C6: 100n, Capacitor_SMD:C_0805_2012Metric, F.Cu at (45.0, 88.5)
- added C7: 470u, Capacitor_THT:CP_Radial_D10.0mm_P5.00mm, F.Cu at (46.4, 81.2)
- added Q2: PMOS, PMOS-SOT23:PMOS-SOT23, F.Cu at (108.5, 106.5)
- added Q3: PMOS, PMOS-SOT23:PMOS-SOT23, F.Cu at (108.5, 111.2)
- added Q4: PMOS, PMOS-SOT23:PMOS-SOT23, F.Cu at (108.5, 116.0)
- added R10: 10k, Resistor_SMD:R_0805_2012Metric, F.Cu at (130.1, 107.0)
- added R3: 100k, Resistor_SMD:R_0805_2012Metric, F.Cu at (130.1, 86.3)
- added R4: 1k, Resistor_SMD:R_0805_2012Metric, F.Cu at (130.1, 89.3)
- added R5: 4k7, Resistor_SMD:R_0805_2012Metric, F.Cu at (130.1, 92.2)
- added R6: 4k7, Resistor_SMD:R_0805_2012Metric, F.Cu at (130.1, 95.2)
- added R7: 10k, Resistor_SMD:R_0805_2012Metric, F.Cu at (130.1, 98.2)
- added R8: 10k, Resistor_SMD:R_0805_2012Metric, F.Cu at (130.1, 101.1)
- added R9: 10k, Resistor_SMD:R_0805_2012Metric, F.Cu at (130.1, 104.0)
- added U3: SMS3.3.TCT, MyESDProtection:SMS3.3.TCT, F.Cu at (146.9, 52.9)
- added U8: SMS3.3.TCT, MyESDProtection:SMS3.3.TCT, F.Cu at (146.9, 57.5)
- moved U7 12.3 mm to (120.8, 37.4)
- moved J2 8.20 mm to (123.5, 65.1)
Connections:
- D3 pad 1: Net-(J1-Pin_2) -> GND
- D3 pad 2: GND -> Net-(J1-Pin_2)

Commit message: IoT update
Parts:
- removed C1: C, Capacitor_SMD:C_0805_2012Metric
- removed L1: 2.2uH, Inductor_SMD:L_0201_0603Metric
- removed Q1: FS8205A, FS8205A:SOP65P640X120-8N
- removed R1: R, Resistor_SMD:R_0805_2012Metric
- removed U4: SC189LSKTRT, SC189LSKTRT:SOT95P280X145-5N
- added C10: 10uF, Capacitor_SMD:C_0805_2012Metric, F.Cu at (62.3, 136.2)
- added C8: 100nF, Capacitor_SMD:C_0805_2012Metric, F.Cu at (62.3, 130.2)
- added C9: 100nF, Capacitor_SMD:C_0805_2012Metric, F.Cu at (62.3, 133.2)
- added J4: Screw_Terminal_01x02, TerminalBlock_Phoenix:TerminalBlock_Phoenix_MPT-0,5-2-2.54_1x02_P2.54mm_Horizontal, F.Cu at (71.5, 120.8)
- added J6: Screw_Terminal_01x02, TerminalBlock_Phoenix:TerminalBlock_Phoenix_MPT-0,5-2-2.54_1x02_P2.54mm_Horizontal, F.Cu at (79.1, 120.8)
- added L2: 2.2uH, Inductor_SMD:L_6.3x6.3_H3, F.Cu at (73.2, 129.4)
- added R11: 4k7, Resistor_SMD:R_0805_2012Metric, F.Cu at (66.8, 121.1)
- added R12: 4k7, Resistor_SMD:R_0805_2012Metric, F.Cu at (66.8, 124.0)
- added R13: 10k, Resistor_SMD:R_0805_2012Metric, F.Cu at (66.8, 127.0)
- added R14: 10k, Resistor_SMD:R_0805_2012Metric, F.Cu at (66.8, 129.9)
- added R15: 10k, Resistor_SMD:R_0805_2012Metric, F.Cu at (66.8, 132.9)
- C2: value 0,1uF -> 10uF
- C3: value 10uF -> 100nF
- J2: value Screw_Terminal_01x02 -> Conn_01x02_Pin; footprint TerminalBlock_Phoenix:TerminalBlock_Phoenix_MPT-0,5-2-2.54_1x02_P2.54mm_Horizontal -> Connector_PinHeader_2.54mm:PinHeader_1x02_P2.54mm_Vertical
- R10: value 10k -> 220
- R4: value 1k -> 220
- U5: value TP4056-42-ESOP8 -> TPS63001; footprint Package_SO:SOIC-8-1EP_3.9x4.9mm_P1.27mm_EP2.41x3.3mm_ThermalVias -> Package_SON:Texas_DRC0010J_ThermalVias
- U6: value TPS63002DRCT -> INA219; footprint TPS63002DRCT:VREG_V62_16624-01YE -> INA219_Module:MODULE_INA219
- moved U1 113.1 mm to (49.7, 110.8)
- moved C6 64.2 mm to (106.0, 68.3)
- moved C7 51.1 mm to (95.5, 67.0)
- moved U8 49.4 mm to (108.5, 88.6)
- moved U3 49.4 mm to (108.5, 84.0)
- moved R10 46.8 mm to (89.7, 83.3)
- moved R3 46.8 mm to (89.7, 62.7)
- moved R4 46.8 mm to (89.7, 65.6)
- moved R5 46.8 mm to (89.7, 68.6)
- moved R6 46.8 mm to (89.7, 71.5)
- moved R7 46.8 mm to (89.7, 74.5)
- moved R8 46.8 mm to (89.7, 77.4)
- moved R9 46.8 mm to (89.7, 80.4)
- moved U5 33.8 mm to (89.9, 129.5)
- moved Q2 32.6 mm to (99.0, 75.3)
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Connections:
- C2 pad 1: Net-(U6-EN) -> LiPo
- C3 pad 1: Net-(U6-VIN) -> Net-(U5-EN)
- C4 pad 1: FB-VOUT -> 3v3
- C5 pad 1: FB-VOUT -> 3v3
- J3 pad 1: VCC -> 3v3
- R10 pad 1: CHG -> Charging
- R10 pad 2: VCC -> Net-(Q5-G)
- R2 pad 1: Net-(U6-VIN) -> LiPo
- R2 pad 2: Net-(U6-EN) -> Net-(U5-EN)
- R4 pad 2: Charging -> Net-(Q5-D)
- R5 pad 1: VCC -> 3v3
- R6 pad 1: VCC -> 3v3
- R7 pad 1: VCC -> 3v3
- R8 pad 1: VCC -> 3v3
- R9 pad 1: FAULT -> Net-(Q5-G)
- R9 pad 2: VCC -> GND
- SunnyBuddy:PRT-12885 pad 7: Net-(J2-Pin_1) -> unconnected-(SunnyBuddy:PRT-12885-LOAD+-Pad7)
- SunnyBuddy:PRT-12885 pad 8: Net-(J2-Pin_2) -> unconnected-(SunnyBuddy:PRT-12885-LOAD--Pad8)
- U1 pad 2: unconnected-(U1-3V3-Pad2) -> 3v3
- U1 pad 8: unconnected-(U1-GPIO0/ADC1_CH0/XTAL_32K_P-Pad8) -> GPIO0
- U2 pad 2: unconnected-(U2-~{INT}-Pad2) -> GPIO0
- U2 pad 5: unconnected-(U2-VSS-Pad5) -> GND
- U2 pad 6: unconnected-(U2-VBACKUP-Pad6) -> Net-(U2-VBACKUP)
- U2 pad 7: unconnected-(U2-VDD-Pad7) -> 3v3
- U2 pad 8: unconnected-(U2-EVI-Pad8) -> Net-(U2-EVI)
- U5 pad 1: unconnected-(U5-TEMP-Pad1) -> 3v3
- U5 pad 2: unconnected-(U5-PROG-Pad2) -> Net-(U5-L2)
- U5 pad 3: unconnected-(U5-GND-Pad3) -> GND
- U5 pad 4: FB-VOUT -> Net-(U5-L1)
- U5 pad 5: unconnected-(U5-BAT-Pad5) -> LiPo
- U5 pad 6: unconnected-(U5-~{STDBY}-Pad6) -> Net-(U5-EN)
- U5 pad 7: unconnected-(U5-~{CHRG}-Pad7) -> Net-(U5-EN)
- U5 pad 8: unconnected-(U5-CE-Pad8) -> Net-(U5-EN)
- U5 pad 9: unconnected-(U5-EPAD-Pad9) -> GND
- U6 pad 1: FB-VOUT -> unconnected-(U6-VCC-Pad1)
- U6 pad 2: Net-(U6-L2) -> unconnected-(U6-GND-Pad2)
- U6 pad 3: GND -> unconnected-(U6-SCL-Pad3)
- U6 pad 4: Net-(U6-L1) -> unconnected-(U6-SDA-Pad4)
- U6 pad 5: Net-(U6-VIN) -> unconnected-(U6-VIN--Pad5)
- U6 pad 6: Net-(U6-EN) -> unconnected-(U6-VIN+-Pad6)
- U7 pad 1: VCC -> 3v3

Commit message: little update
Parts:
- added C1: 22pF, Capacitor_SMD:C_0805_2012Metric, F.Cu at (141.7, 102.1)
- added C11: 22pF, Capacitor_SMD:C_0805_2012Metric, F.Cu at (141.7, 105.1)
- added C12: 100nF, Capacitor_SMD:C_0805_2012Metric, F.Cu at (141.7, 108.2)
- added C14: 100nF, Capacitor_SMD:C_0805_2012Metric, F.Cu at (141.7, 111.2)
- added J7: Conn_01x02_Pin, Connector_PinHeader_2.54mm:PinHeader_1x02_P2.54mm_Vertical, F.Cu at (151.2, 102.9)
- added Q1: PMOS, PMOS-SOT23:PMOS-SOT23, F.Cu at (146.3, 103.2)
- added Q6: PMOS, PMOS-SOT23:PMOS-SOT23, F.Cu at (163.0, 93.0)
- added Q7: PMOS, PMOS-SOT23:PMOS-SOT23, F.Cu at (146.5, 107.5)
- added R1: 4k7, Resistor_SMD:R_0805_2012Metric, F.Cu at (158.2, 93.2)
- added R16: 4k7, Resistor_SMD:R_0805_2012Metric, F.Cu at (158.2, 96.2)
- added R17: 100R, Resistor_SMD:R_0805_2012Metric, F.Cu at (158.2, 99.2)
- added R18: 100R, Resistor_SMD:R_0805_2012Metric, F.Cu at (158.2, 102.1)
- added R19: 10k, Resistor_SMD:R_0805_2012Metric, F.Cu at (158.2, 105.0)
- added R20: 10k, Resistor_SMD:R_0805_2012Metric, F.Cu at (158.2, 108.0)
- added R21: 5k1, Resistor_SMD:R_0805_2012Metric, F.Cu at (141.7, 93.2)
- added R22: 5k1, Resistor_SMD:R_0805_2012Metric, F.Cu at (141.7, 96.2)
- added R23: 1M, Resistor_SMD:R_0805_2012Metric, F.Cu at (141.7, 99.2)
- added R24: 499, Resistor_SMD:R_0805_2012Metric, F.Cu at (146.1, 93.2)
- added R25: 220, Resistor_SMD:R_0805_2012Metric, F.Cu at (146.1, 96.2)
- added R26: 10k, Resistor_SMD:R_0805_2012Metric, F.Cu at (146.1, 99.2)
- added R27: 100k, Resistor_SMD:R_0805_2012Metric, F.Cu at (150.5, 93.2)
- added R28: 10k, Resistor_SMD:R_0805_2012Metric, F.Cu at (150.5, 96.2)
- added R29: 220, Resistor_SMD:R_0805_2012Metric, F.Cu at (150.5, 99.2)
- added R30: 220, Resistor_SMD:R_0805_2012Metric, F.Cu at (169.6, 93.2)
- added R31: 100k, Resistor_SMD:R_0805_2012Metric, F.Cu at (169.6, 96.2)
- added R32: 10k, Resistor_SMD:R_0805_2012Metric, F.Cu at (169.6, 99.2)
- added R33: 220, Resistor_SMD:R_0805_2012Metric, F.Cu at (169.6, 102.1)
- added R34: 4k7, Resistor_SMD:R_0805_2012Metric, F.Cu at (169.6, 105.0)
- added R35: 4k7, Resistor_SMD:R_0805_2012Metric, F.Cu at (169.6, 108.0)
- added SW1: SW_Push, Button_Switch_THT:SW_PUSH_6mm, F.Cu at (215.5, 89.5)
- added SW2: SW_Push, Button_Switch_THT:SW_PUSH_6mm, F.Cu at (215.5, 98.0)
- added U11: PESD5V0L2BT,215, Package_TO_SOT_SMD:SOT-23, F.Cu at (176.6, 94.0)
- added U9: USBLC6-4SC6, Package_TO_SOT_SMD:SOT-23-6, F.Cu at (154.5, 113.5)
- J2: value Conn_01x02_Pin -> USB4085-GF-A_REVA4; footprint Connector_PinHeader_2.54mm:PinHeader_1x02_P2.54mm_Vertical -> USB4085-GF-A_REVA4:GCT_USB4085-GF-A_REVA4
- J4: value Screw_Terminal_01x02 -> Conn_01x04_Pin; footprint TerminalBlock_Phoenix:TerminalBlock_Phoenix_MPT-0,5-2-2.54_1x02_P2.54mm_Horizontal -> Connector_PinHeader_2.54mm:PinHeader_1x04_P2.54mm_Vertical
- J6: value Screw_Terminal_01x02 -> Screw_Terminal_01x04
- moved J2 26.7 mm to (123.3, 105.5)
- moved U1 5.47 mm to (47.0, 115.5)
- moved U6 1.96 mm to (75.5, 105.5)
- moved U7 0.59 mm to (101.5, 50.0)
Connections:
- C10 pad 1: 3v3 -> +3V3
- C2 pad 1: LiPo -> ToDCDC
- C4 pad 1: 3v3 -> +3V3
- C5 pad 1: 3v3 -> +3V3
- C8 pad 1: GND -> +3V3
- C8 pad 2: 3v3 -> GND
- C9 pad 1: 3v3 -> +3V3
- J3 pad 2: SCL -> I2C_SCL
- J3 pad 3: SDA -> I2C_SDA
- J4 pad 2: LiPo -> Net-(J4-Pin_2)
- J6 pad 1: LiPo -> +3V3
- J6 pad 2: GND -> I2C_SCL
- R10 pad 1: Charging -> GPIO21
- R11 pad 1: 3v3 -> +3V3
- R12 pad 1: 3v3 -> +3V3
- R15 pad 1: 3v3 -> +3V3
- R2 pad 1: LiPo -> ToDCDC
- R5 pad 2: SCL -> I2C_SCL
- R6 pad 2: SDA -> I2C_SDA
- U1 pad 10: unconnected-(U1-GPIO8-Pad10) -> GPIO8
- U1 pad 11: unconnected-(U1-GPIO10-Pad11) -> GPIO10
- U1 pad 13: unconnected-(U1-GPIO12/USB_D--Pad13) -> Data-
- U1 pad 14: unconnected-(U1-GPIO13/USB_D+-Pad14) -> Data+
- U1 pad 15: unconnected-(U1-GPIO9-Pad15) -> BOOT
- U1 pad 19: unconnected-(U1-GPIO21-Pad19) -> GPIO21
- U1 pad 2: 3v3 -> +3V3
- U1 pad 20: unconnected-(U1-GPIO22-Pad20) -> CHG
- U1 pad 21: unconnected-(U1-GPIO23-Pad21) -> FAULT
- U1 pad 24: unconnected-(U1-U0RXD/GPIO17-Pad24) -> UART_RX
- U1 pad 25: unconnected-(U1-U0TXD/GPIO16-Pad25) -> UART_TX
- U1 pad 3: unconnected-(U1-EN/CHIP_PU-Pad3) -> RST
- U2 pad 7: 3v3 -> +3V3
- U3 pad 1: SCL -> I2C_SCL
- U3 pad 3: SDA -> I2C_SDA
- U5 pad 1: 3v3 -> +3V3
- U5 pad 10: 3v3 -> +3V3
- U5 pad 5: LiPo -> ToDCDC
- U6 pad 1: unconnected-(U6-VCC-Pad1) -> +3V3
- U6 pad 2: unconnected-(U6-GND-Pad2) -> GND
- U6 pad 3: unconnected-(U6-SCL-Pad3) -> I2C_SCL
- U6 pad 4: unconnected-(U6-SDA-Pad4) -> I2C_SDA
- U6 pad 5: unconnected-(U6-VIN--Pad5) -> Net-(Q6-S)
- U6 pad 6: unconnected-(U6-VIN+-Pad6) -> Load
- U7 pad 1: 3v3 -> +3V3
- U7 pad 3: SCL -> I2C_SCL
- U7 pad 4: SDA -> I2C_SDA
- U7 pad 5: Net-(SunnyBuddy:PRT-12885-Sol+) -> Net-(U4-Sol+)

Commit message: Anemometer update
Parts:
- added J10: Screw_Terminal_01x02, TerminalBlock_RND:TerminalBlock_RND_205-00012_1x02_P5.00mm_Horizontal, F.Cu at (150.5, 74.0)
- added R36: 4k7, Resistor_SMD:R_0805_2012Metric, F.Cu at (131.5, 64.3)
- added R37: 4k7, Resistor_SMD:R_0805_2012Metric, F.Cu at (131.5, 67.3)
- added R38: 220, Resistor_SMD:R_0805_2012Metric, F.Cu at (131.5, 70.2)
- added R39: 10k, Resistor_SMD:R_0805_2012Metric, F.Cu at (135.9, 52.5)
- added R40: 100k, Resistor_SMD:R_0805_2012Metric, F.Cu at (135.9, 55.5)
- added R41: 220, Resistor_SMD:R_0805_2012Metric, F.Cu at (135.9, 58.5)
- added R42: 4k7, Resistor_SMD:R_0805_2012Metric, F.Cu at (135.9, 61.4)
- added R43: 4k7, Resistor_SMD:R_0805_2012Metric, F.Cu at (135.9, 64.3)
- added R44: 220, Resistor_SMD:R_0805_2012Metric, F.Cu at (135.9, 67.3)
- added R45: 10k, Resistor_SMD:R_0805_2012Metric, F.Cu at (135.9, 70.2)
- added R46: 100k, Resistor_SMD:R_0805_2012Metric, F.Cu at (140.4, 52.5)
- added R47: 220, Resistor_SMD:R_0805_2012Metric, F.Cu at (140.4, 55.5)
- added R48: 4k7, Resistor_SMD:R_0805_2012Metric, F.Cu at (140.4, 58.5)
- added R49: 4k7, Resistor_SMD:R_0805_2012Metric, F.Cu at (140.4, 61.4)
- added R5: 220, Resistor_SMD:R_0805_2012Metric, F.Cu at (131.5, 52.5)
- added R50: 220, Resistor_SMD:R_0805_2012Metric, F.Cu at (140.4, 64.3)
- added R51: 10k, Resistor_SMD:R_0805_2012Metric, F.Cu at (140.4, 67.3)
- added R52: 100k, Resistor_SMD:R_0805_2012Metric, F.Cu at (140.4, 70.2)
- added R53: 220, Resistor_SMD:R_0805_2012Metric, F.Cu at (144.8, 52.5)
- added R54: 4k7, Resistor_SMD:R_0805_2012Metric, F.Cu at (144.8, 55.5)
- added R55: 4k7, Resistor_SMD:R_0805_2012Metric, F.Cu at (144.8, 58.5)
- added R56: 20k, Resistor_SMD:R_0805_2012Metric, F.Cu at (144.8, 61.4)
- added R57: 10k, Resistor_SMD:R_0805_2012Metric, F.Cu at (144.8, 64.3)
- added R6: 10k, Resistor_SMD:R_0805_2012Metric, F.Cu at (131.5, 55.5)
- added R7: 100k, Resistor_SMD:R_0805_2012Metric, F.Cu at (131.5, 58.5)
- added R8: 220, Resistor_SMD:R_0805_2012Metric, F.Cu at (131.5, 61.4)
- added U10: PESD5V0L2BT,215, PESD5V0L2BT,215:SOT95P230X110-3N, F.Cu at (150.1, 62.2)
- added U12: PESD5V0L2BT,215, PESD5V0L2BT,215:SOT95P230X110-3N, F.Cu at (150.1, 66.7)
- added U3: PESD5V0L2BT,215, PESD5V0L2BT,215:SOT95P230X110-3N, F.Cu at (150.1, 53.3)
- added U8: PESD5V0L2BT,215, PESD5V0L2BT,215:SOT95P230X110-3N, F.Cu at (150.1, 57.8)
- U11: footprint Package_TO_SOT_SMD:SOT-23 -> PESD5V0L2BT,215:SOT95P230X110-3N

Commit message: External ADC update
Parts:
- removed J10: Screw_Terminal_01x02, TerminalBlock_RND:TerminalBlock_RND_205-00012_1x02_P5.00mm_Horizontal
- removed J3: Conn_01x05_Pin, Connector_PinSocket_2.54mm:PinSocket_1x05_P2.54mm_Vertical
- removed J5: Conn_01x04_Pin, Connector_PinSocket_2.54mm:PinSocket_1x04_P2.54mm_Vertical
- removed J6: Screw_Terminal_01x04, TerminalBlock_Phoenix:TerminalBlock_Phoenix_MPT-0,5-2-2.54_1x02_P2.54mm_Horizontal
- removed J7: Conn_01x02_Pin, Connector_PinHeader_2.54mm:PinHeader_1x02_P2.54mm_Vertical
- removed R1, R11, R12, R16, R36, R37, R42, R43, R48, R49, R54, R55: 4k7, Resistor_SMD:R_0805_2012Metric
- removed R30: 220, Resistor_SMD:R_0805_2012Metric
- removed R31: 100k, Resistor_SMD:R_0805_2012Metric
- removed the R5 at (89.7, 68.6)
- removed the R5 at (131.5, 52.5)
- removed R56: 20k, Resistor_SMD:R_0805_2012Metric
- removed R57: 10k, Resistor_SMD:R_0805_2012Metric
- removed the R6 at (131.5, 55.5)
- removed the R6 at (89.7, 71.5)
- removed the R7 at (89.7, 74.5)
- removed the R7 at (131.5, 58.5)
- removed the R8 at (131.5, 61.4)
- removed the R8 at (89.7, 77.4)
- removed SunnyBuddy:PRT-12885: ~, SunnyBuddy:PRT-12885
- removed the U3 at (150.1, 53.3)
- removed the U3 at (108.5, 84.0)
- removed the U8 at (150.1, 57.8)
- removed the U8 at (108.5, 88.6)
- added C13: 100nF, Capacitor_SMD:C_0805_2012Metric, F.Cu at (95.7, 101.6)
- added D2: STS321050B100-EA, Diode_SMD:D_SOD-323, F.Cu at (95.7, 104.6)
- added J11: Screw_Terminal_01x03, TerminalBlock_Phoenix:TerminalBlock_Phoenix_MKDS-1-3-3.81_1x03_P3.81mm_Horizontal, F.Cu at (73.3, 119.0)
- added JP1: Jumper_2_Open, TestPoint:TestPoint_2Pads_Pitch2.54mm_Drill0.8mm, F.Cu at (40.5, 87.0)
- added R5: 220, Resistor_SMD:R_0805_2012Metric, F.Cu at (72.6, 95.1)
- added R58: 220, Resistor_SMD:R_0805_2012Metric, F.Cu at (81.4, 112.8)
- added R59: 10k, Resistor_SMD:R_0805_2012Metric, F.Cu at (85.8, 95.1)
- added R6: 10k, Resistor_SMD:R_0805_2012Metric, F.Cu at (72.6, 98.1)
- added R60: 100k, Resistor_SMD:R_0805_2012Metric, F.Cu at (85.8, 98.1)
- added R61: 220, Resistor_SMD:R_0805_2012Metric, F.Cu at (85.8, 101.0)
- added R7: 100k, Resistor_SMD:R_0805_2012Metric, F.Cu at (72.6, 101.0)
- added R8: 220, Resistor_SMD:R_0805_2012Metric, F.Cu at (72.6, 104.0)
- added U13: MCP3422A0-E/SN, MCP3422A7ESN:SOIC127P600X175-8N, F.Cu at (92.9, 96.9)
- added U3: PESD5V0L2BT,215, PESD5V0L2BT,215:SOT95P230X110-3N, F.Cu at (91.1, 102.3)
- added U4: SunnyBuddy:PRT-12885, SunnyBuddy:PRT-12885, F.Cu at (48.9, 23.9)
- added U8: PESD5V0L2BT,215, PESD5V0L2BT,215:SOT95P230X110-3N, F.Cu at (91.1, 106.8)
- D3: value ~ -> SMBJ24CA:DO214AA
- R17, R18: value 100R -> 4k7
- R32: value 10k -> 220
- R33: value 220 -> 10k
- R34: value 4k7 -> 100k
- R35: value 4k7 -> 220
- moved SW1 169.2 mm to (47.6, 110.4)
- moved SW2 169.2 mm to (47.6, 119.0)
- moved R32 97.3 mm to (72.6, 106.9)
- moved R33 97.3 mm to (72.6, 109.9)
- moved R34 97.3 mm to (72.6, 112.8)
- moved J2 95.5 mm to (30.4, 127.8)
- moved R21 94.9 mm to (47.8, 106.9)
- moved R24 94.2 mm to (52.2, 101.0)
- moved R25 94.2 mm to (52.2, 104.0)
- moved R26 94.2 mm to (52.2, 106.9)
- moved R27 93.9 mm to (56.6, 95.1)
- moved R28 93.9 mm to (56.6, 98.1)
- moved R29 93.9 mm to (56.6, 101.0)
- moved R35 93.5 mm to (77.0, 95.1)
- moved U9 90.9 mm to (64.9, 128.9)
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Connections:
- net Net-(Q4-D) renamed Vin+
- R32 pad 1: GND -> GPIO11
- R32 pad 2: Net-(Q8-G) -> Net-(Q10-G)
- R33 pad 1: Net-(Q8-D) -> GND
- R33 pad 2: Net-(Q9-G) -> Net-(Q10-G)
- R34 pad 1: I2C_SCL -> Net-(Q10-D)
- R35 pad 1: I2C_SDA -> Net-(Q10-D)
- R35 pad 2: +3V3 -> Net-(Q11-G)
- R38 pad 1: GPIO10 -> GPIO15
- R44 pad 1: GPIO10 -> GPIO18
- R50 pad 1: GPIO10 -> GPIO19
- U1 pad 12: unconnected-(U1-GPIO11-Pad12) -> GPIO12
- U1 pad 16: unconnected-(U1-GPIO18-Pad16) -> GPIO18
- U1 pad 17: unconnected-(U1-GPIO19-Pad17) -> GPIO19
- U1 pad 18: unconnected-(U1-GPIO20-Pad18) -> GPIO20
- U1 pad 23: unconnected-(U1-GPIO15-Pad23) -> GPIO15
- U7 pad 5: Net-(U4-Sol+) -> Vin-

Commit message: Tomáš update
Parts:
- removed C1: 22pF, Capacitor_SMD:C_0805_2012Metric
- removed JP1: Jumper_2_Open, TestPoint:TestPoint_2Pads_Pitch2.54mm_Drill0.8mm
- removed R13, R14: 10k, Resistor_SMD:R_0805_2012Metric
- added C15: 1nF, Capacitor_SMD:C_0805_2012Metric, F.Cu at (69.8, 128.0)
- added C16: 10uF, Capacitor_SMD:C_0805_2012Metric, F.Cu at (134.3, 58.1)
- added C17: 1uF, Capacitor_SMD:C_0805_2012Metric, F.Cu at (134.3, 61.1)
- added C18: 100nF, Capacitor_SMD:C_0805_2012Metric, F.Cu at (134.3, 64.1)
- added C19: 100nF, Capacitor_SMD:C_0805_2012Metric, F.Cu at (134.3, 67.1)
- added Q10: NMOS, NMOS:SOT95P230X110-3N, F.Cu at (111.9, 44.9)
- added Q11: NMOS, NMOS:SOT95P230X110-3N, F.Cu at (117.3, 36.0)
- added Q12: NMOS, NMOS:SOT95P230X110-3N, F.Cu at (117.3, 40.4)
- added Q13: NMOS, NMOS:SOT95P230X110-3N, F.Cu at (117.3, 44.9)
- added Q14: NMOS, NMOS:SOT95P230X110-3N, F.Cu at (122.6, 36.0)
- added Q15: NMOS, NMOS:SOT95P230X110-3N, F.Cu at (122.6, 40.4)
- added Q16: NMOS, NMOS:SOT95P230X110-3N, F.Cu at (122.6, 44.9)
- added Q17: NMOS, NMOS:SOT95P230X110-3N, F.Cu at (127.9, 36.0)
- added Q18: NMOS, NMOS:SOT95P230X110-3N, F.Cu at (127.9, 40.4)
- added Q19: NMOS, NMOS:SOT95P230X110-3N, F.Cu at (127.9, 44.9)
- added Q5: NMOS, NMOS:SOT95P230X110-3N, F.Cu at (42.4, 94.3)
- added Q8: NMOS, NMOS:SOT95P230X110-3N, F.Cu at (111.9, 36.0)
- added Q9: NMOS, NMOS:SOT95P230X110-3N, F.Cu at (111.9, 40.4)
- added R30: 100, Resistor_SMD:R_0805_2012Metric, F.Cu at (63.6, 110.0)
- C11: value 22pF -> 1uF
- R24: value 499 -> 100
- R33, R39, R45, R51, R59, R6: value 10k -> 100k
- moved U3 60.5 mm to (129.7, 55.8)
- moved U8 60.5 mm to (129.7, 60.2)
- moved C13 60.5 mm to (134.3, 55.1)
- moved J11 60.5 mm to (111.9, 72.5)
- moved R38 60.5 mm to (115.6, 51.5)
- moved R39 60.5 mm to (115.6, 54.5)
- moved R47 60.5 mm to (120.0, 51.5)
- moved R50 60.5 mm to (120.0, 54.5)
- moved R6 60.5 mm to (111.2, 51.5)
- moved R60 60.5 mm to (124.4, 51.5)
- moved R61 60.5 mm to (124.4, 54.5)
- moved R7 60.5 mm to (111.2, 54.5)
- moved U10 60.5 mm to (129.7, 64.7)
- moved U11 60.5 mm to (129.7, 69.1)
- moved U12 60.5 mm to (129.7, 73.6)
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Connections:
- C11 pad 1: Data- -> +3V3
- J2 pad S1: Net-(J2-SHELL-PadS1) -> Net-(C15-Pad1)
- J2 pad S2: Net-(J2-SHELL-PadS1) -> Net-(C15-Pad1)
- J2 pad S3: Net-(J2-SHELL-PadS1) -> Net-(C15-Pad1)
- J2 pad S4: Net-(J2-SHELL-PadS1) -> Net-(C15-Pad1)
- J4 pad 3: UART_RX -> Net-(J4-Pin_3)
- R23 pad 1: Net-(J2-SHELL-PadS1) -> GND
- R23 pad 2: GND -> Net-(C15-Pad1)
- R27 pad 2: Net-(JP1-B) -> GPIO8
- U2 pad 6: Net-(U2-VBACKUP) -> +3V3
- U2 pad 8: Net-(U2-EVI) -> unconnected-(U2-EVI-Pad8)

Commit message: little update
Parts:
- removed J11: Screw_Terminal_01x03, TerminalBlock_Phoenix:TerminalBlock_Phoenix_MKDS-1-3-3.81_1x03_P3.81mm_Horizontal
- added J10: Screw_Terminal_01x04, TerminalBlock_Phoenix:TerminalBlock_Phoenix_MKDS-1,5-4-5.08_1x04_P5.08mm_Horizontal, F.Cu at (113.3, 145.5)
- added J3: Screw_Terminal_01x04, TerminalBlock_Phoenix:TerminalBlock_Phoenix_MKDS-1,5-4-5.08_1x04_P5.08mm_Horizontal, F.Cu at (113.3, 97.0)
- added J5: Screw_Terminal_01x04, TerminalBlock_Phoenix:TerminalBlock_Phoenix_MKDS-1,5-4-5.08_1x04_P5.08mm_Horizontal, F.Cu at (113.3, 109.1)
- added J6: Screw_Terminal_01x04, TerminalBlock_Phoenix:TerminalBlock_Phoenix_MKDS-1,5-4-5.08_1x04_P5.08mm_Horizontal, F.Cu at (113.3, 121.2)
- added J7: Screw_Terminal_01x02, TerminalBlock_Phoenix:TerminalBlock_Phoenix_MKDS-1,5-2-5.08_1x02_P5.08mm_Horizontal, F.Cu at (154.9, 109.1)
- added J8: Screw_Terminal_01x04, TerminalBlock_Phoenix:TerminalBlock_Phoenix_MKDS-1,5-4-5.08_1x04_P5.08mm_Horizontal, F.Cu at (113.3, 133.4)
- added J9: Screw_Terminal_01x03, TerminalBlock_Phoenix:TerminalBlock_Phoenix_MKDS-1,5-3-5.08_1x03_P5.08mm_Horizontal, F.Cu at (136.8, 97.0)
- J1: footprint TerminalBlock_Phoenix:TerminalBlock_Phoenix_MPT-0,5-2-2.54_1x02_P2.54mm_Horizontal -> TerminalBlock_Phoenix:TerminalBlock_Phoenix_MKDS-1,5-2-5.08_1x02_P5.08mm_Horizontal
- moved J1 120.7 mm to (154.9, 97.0)
Connections:
- C7 pad 1: Net-(J1-Pin_2) -> Net-(J7-Pin_2)
- D3 pad 2: Net-(J1-Pin_2) -> Net-(J7-Pin_2)
- J1 pad 1: GND -> Load
- J1 pad 2: Net-(J1-Pin_2) -> GND
- Q2 pad 3: Net-(J1-Pin_2) -> Net-(J7-Pin_2)
