File: Hardware/hw/hw.kicad_pcb (KiCad board)
At the start: 2 copper layers, 109 parts, among them J1 Screw_Terminal_01x02, J10 Screw_Terminal_01x04, J2 USB4085-GF-A_REVA4, J3 Screw_Terminal_01x04, J4 Conn_01x04_Pin, J5 Screw_Terminal_01x04, J6 Screw_Terminal_01x04, J7 Screw_Terminal_01x02, J8 Screw_Terminal_01x04, J9 Screw_Terminal_01x03, Q1 PMOS, Q10 NMOS, Q11 NMOS, Q12 NMOS, Q13 NMOS, Q14 NMOS, Q15 NMOS, Q16 NMOS, Q17 NMOS, Q18 NMOS, Q19 NMOS, Q2 PMOS, Q3 PMOS, Q4 PMOS, Q5 NMOS, Q6 PMOS, Q7 PMOS, Q8 NMOS, Q9 NMOS, SW1 SW_Push, SW2 SW_Push, U1 ESP32-C6-WROOM-1, U10 PESD5V0L2BT,215, U11 PESD5V0L2BT,215, U12 PESD5V0L2BT,215, U13 MCP3422A0-E/SN, U2 RV-3028-C7, U3 PESD5V0L2BT,215, U4 SunnyBuddy:PRT-12885, U5 TPS63001, U6 INA219, U7 INA219, U8 PESD5V0L2BT,215, U9 USBLC6-4SC6

Commit message: HW update
Parts:
- U4: renamed from U1; footprint PCM_Espressif:ESP32-C6-WROOM-1 -> PCM_Espressif:ESP32-C6-WROOM-1U
- moved C2 146.3 mm to (195.8, 73.1)
- moved C10 142.8 mm to (206.1, 101.1)
- moved C11 142.8 mm to (210.6, 98.1)
- moved C12 142.8 mm to (206.1, 104.1)
- moved C13 142.8 mm to (210.6, 104.1)
- moved C3 142.8 mm to (206.1, 92.0)
- moved C4 142.8 mm to (206.1, 95.1)
- moved C5 142.8 mm to (210.6, 101.1)
- moved C6 142.8 mm to (210.6, 92.0)
- moved C7 142.8 mm to (210.6, 95.1)
- moved C8 142.8 mm to (206.1, 98.1)
- moved C9 142.8 mm to (206.1, 107.1)
- moved D1 142.8 mm to (184.5, 65.4)
- moved J3 142.8 mm to (208.9, 78.1)
- moved L1 142.8 mm to (208.2, 112.5)
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- renumbered C7 to C1, C5 to C10, C12 to C11, C8 to C12, C15 to C13, C19 to C14, C16 to C15, C17 to C16, C18 to C17, C13 to C18, C6 to C2, C2 to C3, C3 to C4, C14 to C5, C10 to C6, C11 to C7, C4 to C8, D3 to D1, J7 to J1, J9 to J10, J1 to J2, J4 to J3, J2 to J4, J10 to J5, J3 to J6, J5 to J7, J6 to J8, J8 to J9, L2 to L1, Q2 to Q1, Q12 to Q10, Q9 to Q11, Q11 to Q12, Q16 to Q15, Q15 to Q16, Q3 to Q2, Q5 to Q3, Q6 to Q5, Q7 to Q6, Q1 to Q7, Q10 to Q9, R10 to R1, R28 to R10, R29 to R11, R27 to R12, R17 to R13, R18 to R14, R30 to R15, R24 to R16, R21 to R17, R22 to R18, R23 to R19, R9 to R2, R15 to R20, R5 to R21, R32 to R22, R38 to R23, R6 to R24, R33 to R25, R39 to R26, R7 to R27, R34 to R28, R40 to R29, R8 to R30, R35 to R31, R41 to R32, R44 to R33, R50 to R34, R45 to R35, R51 to R36, R46 to R37, R52 to R38, R47 to R39, R53 to R40, R58 to R41, R59 to R42, R60 to R43, R61 to R44, R19 to R5, R20 to R6, R2 to R7, R26 to R8, R25 to R9, SW2 to SW1, SW1 to SW2, U7 to U1, U11 to U10, U10 to U11, U6 to U2, U4 to U3, U9 to U6, U2 to U7, U3 to U8, U8 to U9
Other:
- copper layers 2 -> 4

Commit message: Mega update
Parts:
- moved Q3 124.7 mm to (75.2, 138.2)
- moved U7 121.6 mm to (240.8, 114.2), turned to 0 degrees
- moved Q17 115.1 mm to (171.4, 142.6), turned to 90 degrees
- moved Q18 115.1 mm to (189.6, 137.6), turned to 90 degrees
- moved C2 113.0 mm to (87.6, 105.6)
- moved Q19 112.0 mm to (182.8, 142.5), turned to -90 degrees
- moved Q14 110.3 mm to (149.3, 143.0), turned to 90 degrees
- moved R44 108.1 mm to (186.9, 142.6), turned to 90 degrees
- moved R42 107.6 mm to (189.7, 134.1), turned to 180 degrees
- moved R43 106.1 mm to (178.8, 142.6), turned to -90 degrees
- moved Q15 105.7 mm to (162.3, 142.8), turned to -90 degrees
- moved Q16 104.1 mm to (140.7, 142.9), turned to -90 degrees
- moved R41 103.7 mm to (190.3, 142.6), turned to 90 degrees
- moved U13 100.8 mm to (183.3, 136.7)
- moved D1 100.0 mm to (89.6, 96.8)
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Connections:
- U4 pad 12: GPIO12 -> GPIO11

Commit message: new PCB
Parts:
- moved R18 167.1 mm to (69.2, 102.5), turned to 90 degrees
- moved R19 163.8 mm to (72.5, 102.5), turned to -90 degrees
- moved U6 153.7 mm to (79.7, 107.9), turned to 90 degrees
- moved R16 153.4 mm to (78.9, 97.9)
- moved R15 153.4 mm to (78.9, 94.5)
- moved R11 152.7 mm to (76.2, 130.5), turned to -90 degrees
- moved R9 152.0 mm to (76.2, 119.0), turned to -90 degrees
- moved R10 150.1 mm to (79.2, 130.5), turned to 90 degrees
- moved SW2 149.3 mm to (66.7, 130.3)
- moved R8 149.3 mm to (79.2, 119.0), turned to 90 degrees
- moved SW1 149.1 mm to (66.8, 118.8)
- moved Q6 148.4 mm to (79.7, 102.5), turned to 90 degrees
- moved Q7 148.1 mm to (79.7, 113.3), turned to 90 degrees
- moved C13 136.6 mm to (75.7, 102.5), turned to 90 degrees
- moved C11 135.4 mm to (77.5, 135.3)
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
Commit message: update
Parts:
- moved U4 3.27 mm to (125.8, 119.1)
- moved Q7 2.43 mm to (77.2, 113.6)
- moved U6 2.43 mm to (77.2, 108.2)
- moved J4 1.81 mm to (67.8, 110.8)
- moved C7 1.57 mm to (111.5, 117.8)
- moved C9 1.57 mm to (111.6, 111.0)
- moved R12 1.57 mm to (111.4, 128.4)
- moved R13 1.57 mm to (111.4, 121.5)
- moved R14 1.57 mm to (111.5, 125.0)
- moved C6 1.57 mm to (111.5, 114.3)
- moved D1 1.27 mm to (124.4, 88.7)
- moved C1 0.20 mm to (130.7, 88.5)
Routing:
- net Vin+: track 0.00 -> 61.6 mm, vias 0 -> 3
- net Net-(J1-Pin_2): track 0.00 -> 29.9 mm
- net +3V3: track 0.00 -> 23.6 mm, vias 0 -> 2
- net Net-(Q4-G): track 0.00 -> 16.5 mm, vias 0 -> 2
- net Net-(Q2-S): track 0.00 -> 15.7 mm
- net Net-(Q3-G): track 0.00 -> 14.4 mm, vias 0 -> 2
- net Net-(U5-EN): track 0.00 -> 13.1 mm, vias 0 -> 3
- net Net-(U5-L1): track 0.00 -> 11.8 mm
- net Net-(U5-L2): track 0.00 -> 11.7 mm
- net Net-(Q3-D): track 0.00 -> 8.05 mm
- net ToDCDC: track 0.00 -> 8.01 mm
- net Net-(Q1-D): track 0.00 -> 5.76 mm
- net CHG: track 0.00 -> 3.37 mm
- net FAULT: track 0.00 -> 3.22 mm
- added copper zone on B.Cu, net GND
- added copper zone on F.Cu, net GND
- added copper zone on In1.Cu, net GND
- added copper zone on In2.Cu, net GND
Other:
- board outline added: 128.2 x 76.5 mm

Commit message: ...
Routing:
- net +3V3: track 23.6 -> 446.0 mm, vias 2 -> 18
- net I2C_SDA: track 0.00 -> 280.5 mm, vias 0 -> 4
- net I2C_SCL: track 0.00 -> 278.8 mm, vias 0 -> 3
- net Load: track 0.00 -> 114.9 mm
- net Vin-: track 0.00 -> 86.1 mm
- net UART_TX: track 0.00 -> 79.7 mm, vias 0 -> 3
- net UART_RX: track 0.00 -> 76.3 mm, vias 0 -> 3
- net BOOT: track 0.00 -> 71.4 mm, vias 0 -> 4
- net GPIO20: track 0.00 -> 66.9 mm, vias 0 -> 2
- net ToDCDC: track 8.01 -> 74.0 mm, vias 0 -> 2
- net Data-: track 0.00 -> 61.4 mm, vias 0 -> 2
- net Data+: track 0.00 -> 60.6 mm, vias 0 -> 2
- net GPIO10: track 0.00 -> 55.3 mm, vias 0 -> 4
- net GPIO19: track 0.00 -> 53.5 mm, vias 0 -> 2
- net RST: track 0.00 -> 48.8 mm, vias 0 -> 2
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
Commit message: Hardware v1.0
Parts:
- added H1: MountingHole, MountingHole:MountingHole_3.2mm_M3_DIN965_Pad_TopBottom, F.Cu at (190.9, 89.7)
- added H2: MountingHole, MountingHole:MountingHole_3.2mm_M3_DIN965_Pad_TopBottom, F.Cu at (88.0, 133.5)
Routing:
- net GND: track 19.4 -> 15.2 mm, vias 3 -> 4
- net ToDCDC: track 74.0 -> 69.9 mm, vias 2 -> 4
- net Net-(U5-EN): track 19.2 -> 16.1 mm
- net +3V3: track 446.0 -> 443.3 mm, vias 18 -> 19
- net Net-(U5-L1): track 13.7 -> 11.1 mm
- net Net-(U5-L2): track 13.8 -> 11.8 mm, vias 2 -> 0
- net FAULT: track 25.4 -> 26.0 mm
- net RST: track 48.8 -> 48.9 mm, vias 2 -> 4
- net GPIO11: vias 0 -> 2
- net Vin-: vias 0 -> 1
Other:
- board size 128.2 x 76.5 mm -> 130.8 x 77.2 mm
- board text added: "ADC"
- board text added: "Author: Peter Kolok Year: 2026 Rev: Tomáš Bača Version: 1.0"
- board text added: "BAT+"
- board text added: "BAT-"
- board text added: "GND"
- board text added: "RX"
- board text added: "SCL"
- board text added: "SDA"
- board text added: "Sol+"
- board text added: "Sol-"
- board text added: "TX"
- board text added: "VCC"

Commit message: Stupid-Stupid update
Parts:
- Q9: footprint NMOS:SOT95P230X110-3N -> NMOS:AO3400A
Routing:
- net Net-(J1-Pin_2): track 47.4 -> 40.5 mm
Changed lines of the file:
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@@
 		)
 	)
-	(footprint "NMOS:SOT95P230X110-3N"
+	(footprint "NMOS:AO3400A"
 		(layer "F.Cu")
 		(at 105.55 142.97 90)
 		(property "Reference" "Q9"
-			(at -0.03 2.2 90)
+			(at 1.315 -3.335 90)
 			(layer "F.SilkS")
 			(effects
 				(font
-					(size 0.5 0.5)
+					(size 1 1)
 					(thickness 0.15)
 				)
@@
 		)
 		(property "Value" "NMOS"
-			(at 8.3 3.335 90)
+			(at 3.7 2.9 90)
 			(layer "F.Fab")
 			(effects
@@
 			(layer "F.SilkS")
 		)
-		(fp_circle
-			(center -2.25 -0.975)
-			(end -2.15 -0.975)
-			(stroke
-				(width 0.2)
-				(type solid)
-			)
-			(fill no)
-			(layer "F.SilkS")
-		)
 		(fp_line
 			(start 1.86 -1.7)
@@
 			(layer "F.Fab")
 		)
-		(fp_circle
-			(center -2.25 -0.975)
-			(end -2.15 -0.975)
-			(stroke
-				(width 0.2)
-				(type solid)
-			)
-			(fill no)
-			(layer "F.Fab")
-		)
 		(pad "1" smd roundrect
-			(at -0.98 -0.95 90)
+			(at 0.98 0 90)
 			(size 1.26 0.59)
 			(layers "F.Cu" "F.Mask" "F.Paste")
@@
 		)
 		(pad "2" smd roundrect
-			(at -0.98 0.95 90)
+			(at -0.98 -0.95 90)
 			(size 1.26 0.59)
 			(layers "F.Cu" "F.Mask" "F.Paste")
@@
 		)
 		(pad "3" smd roundrect
-			(at 0.98 0 90)
+			(at -0.98 0.95 90)
 			(size 1.26 0.59)
 			(layers "F.Cu" "F.Mask" "F.Paste")
@@
 		(width 1)
 		(layer "F.Cu")
-		(net 3)
-	)
-	(segment
-		(start 110.3 96.15)
-		(end 110.3 89.2425)
-		(width 1)
-		(layer "F.Cu")

Commit message: RTC update
Parts:
- added R45: 10k, Resistor_SMD:R_0805_2012Metric, F.Cu at (118.7, 132.8)
- added R46: 10k, Resistor_SMD:R_0805_2012Metric, F.Cu at (114.8, 132.8)
- L1: footprint Inductor_SMD:L_6.3x6.3_H3 -> Inductor_SMD:L_Taiyo-Yuden_NR-60xx
- Q10, Q11, Q12, Q13, Q14, Q15, Q16, Q17, Q18, Q19, Q3, Q8: footprint NMOS:SOT95P230X110-3N -> NMOS:AO3400A
Connections:
- U7 pad 6: +3V3 -> Net-(U7-VBACKUP)
- U7 pad 8: unconnected-(U7-EVI-Pad8) -> Net-(U7-EVI)
Routing:
- net +3V3: track 443.3 -> 8.02 mm, vias 19 -> 0
- net I2C_SDA: track 280.5 -> 0.00 mm, vias 4 -> 0
- net I2C_SCL: track 278.8 -> 0.00 mm, vias 3 -> 0
- net Load: track 114.9 -> 0.00 mm
- net Vin-: track 86.1 -> 0.00 mm, vias 1 -> 0
- net UART_TX: track 79.7 -> 0.00 mm, vias 3 -> 0
- net UART_RX: track 76.3 -> 0.00 mm, vias 3 -> 0
- net Vin+: track 74.7 -> 0.00 mm, vias 3 -> 0
- net BOOT: track 71.4 -> 0.00 mm, vias 4 -> 0
- net ToDCDC: track 69.9 -> 0.00 mm, vias 4 -> 0
- net GPIO20: track 66.9 -> 0.00 mm, vias 2 -> 0
- net Data-: track 61.4 -> 0.00 mm, vias 2 -> 0
- net Data+: track 60.6 -> 0.00 mm, vias 2 -> 0
- net GPIO10: track 55.3 -> 0.00 mm, vias 4 -> 0
- net GPIO19: track 53.5 -> 0.00 mm, vias 2 -> 0
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- removed copper zone on In1.Cu, net GND
- removed copper zone on In2.Cu, net GND
Other:
- copper layers 4 -> 2
