File: Hardware/hw/hw.kicad_pcb (KiCad board)
At the start: 2 copper layers, 130.8 x 77.2 mm, 113 parts, among them J1 Screw_Terminal_01x02, J10 Screw_Terminal_01x03, J2 Screw_Terminal_01x02, J3 Conn_01x04_Pin, J4 USB4085-GF-A_REVA4, J5 Screw_Terminal_01x04, J6 Screw_Terminal_01x04, J7 Screw_Terminal_01x04, J8 Screw_Terminal_01x04, J9 Screw_Terminal_01x04, Q1 PMOS, Q10 NMOS, Q11 NMOS, Q12 NMOS, Q13 NMOS, Q14 NMOS, Q15 NMOS, Q16 NMOS, Q17 NMOS, Q18 NMOS, Q19 NMOS, Q2 PMOS, Q3 NMOS, Q4 PMOS, Q5 PMOS, Q6 PMOS, Q7 PMOS, Q8 NMOS, Q9 NMOS, SW1 SW_Push, SW2 SW_Push, U1 INA219, U10 PESD5V0L2BT,215, U11 PESD5V0L2BT,215, U12 PESD5V0L2BT,215, U13 MCP3422A0-E/SN, U2 INA219, U3 SunnyBuddy:PRT-12885, U4 ESP32-C6-WROOM-1, U5 TPS63001, U6 USBLC6-4SC6, U7 RV-3028-C7, U8 PESD5V0L2BT,215, U9 PESD5V0L2BT,215

Commit message: home work
Routing:
- net +3V3: track 8.02 -> 71.4 mm, vias 0 -> 4
- net GPIO0: track 0.00 -> 31.4 mm
- net I2C_SCL: track 0.00 -> 30.4 mm, vias 0 -> 2
- net I2C_SDA: track 0.00 -> 29.9 mm, vias 0 -> 2
- net ToDCDC: track 0.00 -> 20.2 mm
- net Net-(U5-EN): track 0.00 -> 18.1 mm
- net Net-(U5-L1): track 0.00 -> 13.7 mm, vias 0 -> 2
- net Net-(U5-L2): track 0.00 -> 9.90 mm, vias 0 -> 2
- net GPIO8: track 0.00 -> 8.71 mm
- net GND: vias 0 -> 2

Commit message: Screw matrix update
Parts:
- added J11: KF301-2P, KF301-2P:HANDSON_KF301-2P, F.Cu at (50.3, 105.3)
- J1: footprint TerminalBlock_Phoenix:TerminalBlock_Phoenix_MKDS-1,5-2-5.08_1x02_P5.08mm_Horizontal -> TerminalBlock_Phoenix:TerminalBlock_Phoenix_MKDS-1,5-2_1x02_P5.00mm_Horizontal
- J10: value Screw_Terminal_01x03 -> Screw_Terminal_01x02; footprint TerminalBlock_Phoenix:TerminalBlock_Phoenix_MKDS-1,5-3-5.08_1x03_P5.08mm_Horizontal -> TerminalBlock_Phoenix:TerminalBlock_Phoenix_MKDS-1,5-2_1x02_P5.00mm_Horizontal
- J2: value Screw_Terminal_01x02 -> Screw_Terminal_01x03; footprint TerminalBlock_Phoenix:TerminalBlock_Phoenix_MKDS-1,5-2-5.08_1x02_P5.08mm_Horizontal -> TerminalBlock_Phoenix:TerminalBlock_Phoenix_MKDS-1,5-3_1x03_P5.00mm_Horizontal
- J5, J6, J7, J8, J9: footprint TerminalBlock_Phoenix:TerminalBlock_Phoenix_MKDS-1,5-4-5.08_1x04_P5.08mm_Horizontal -> TerminalBlock_Phoenix:TerminalBlock_Phoenix_MKDS-1,5-4_1x04_P5.00mm_Horizontal
- moved J2 125.9 mm to (177.1, 151.9), turned to 0 degrees
- moved J10 125.3 mm to (70.4, 86.0), turned to -90 degrees
- moved J1 0.22 mm to (116.8, 88.2)
Connections:
- J10 pad 1: +3V3 -> Load
- J10 pad 2: ADC -> GND
- J2 pad 1: Load -> +3V3
- J2 pad 2: GND -> ADC
- Q19 pad 1: Net-(J10-Pin_3) -> Net-(J2-Pin_3)

Commit message: PCB update
Parts:
- removed D2: STS321050B100-EA, Diode_SMD:D_SOD-323
- removed J11: KF301-2P, KF301-2P:HANDSON_KF301-2P
- added D3: 1N4448W, Diode_SMD:D_SOD-123, F.Cu at (173.1, 145.8)
- moved H1 114.9 mm to (84.6, 133.2)
- moved H2 50.4 mm to (130.1, 105.7)
- moved U1 26.3 mm to (92.9, 92.7), turned to 0 degrees
- moved C2 24.8 mm to (114.3, 104.5), turned to -90 degrees
- moved U2 24.4 mm to (92.8, 117.4), turned to 180 degrees
- moved R46 22.2 mm to (92.8, 135.3)
- moved R45 21.8 mm to (97.0, 135.4)
- moved U7 20.6 mm to (102.5, 135.6)
- moved C12 19.9 mm to (107.3, 135.4), turned to 90 degrees
- moved R20 18.9 mm to (111.8, 135.4)
- moved Q10 17.6 mm to (110.0, 146.2)
- moved U10 15.8 mm to (126.1, 145.8)
- moved C4 15.4 mm to (131.1, 113.1), turned to 90 degrees
- moved Q3 13.6 mm to (138.1, 98.5)
- moved R7 12.4 mm to (112.9, 112.9), turned to -90 degrees
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Routing:
- net Load: track 0.00 -> 120.7 mm
- net Vin-: track 0.00 -> 77.9 mm
- net ToDCDC: track 20.2 -> 67.1 mm, vias 0 -> 2
- net Vin+: track 0.00 -> 39.9 mm, vias 0 -> 4
- net Net-(J1-Pin_2): track 0.00 -> 35.3 mm
- net GPIO0: track 31.4 -> 0.00 mm
- net +3V3: track 71.4 -> 40.3 mm, vias 4 -> 2
- net I2C_SCL: track 30.4 -> 0.00 mm, vias 2 -> 0
- net I2C_SDA: track 29.9 -> 0.00 mm, vias 2 -> 0
- net Net-(Q4-G): track 0.00 -> 18.5 mm, vias 0 -> 2
- net Net-(J3-Pin_4): track 0.00 -> 17.4 mm
- net Net-(Q2-S): track 0.00 -> 13.3 mm
- net Net-(U7-VBACKUP): track 13.0 -> 0.00 mm, vias 2 -> 0
- net VBUS: track 0.00 -> 12.6 mm
- net Net-(Q3-D): track 0.00 -> 11.3 mm
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Other:
- board size 130.8 x 77.2 mm -> 130.6 x 81.9 mm
- board text removed: "Author: Peter Kolok Year: 2026 Rev: Tomáš Bača Version: 1.0"
- board text removed: "BAT+"
- board text removed: "BAT-"
- board text removed: "RX"
- board text removed: "Sol+"
- board text removed: "Sol-"
- board text removed: "TX"
