File: Hardware/hw/charging.kicad_sch (KiCad schematic)
At the start: 19 parts, among them J1 Screw_Terminal_01x02, J2 Screw_Terminal_01x02, Q1 PMOS, Q2 PMOS, Q3 NMOS, Q4 PMOS, Q5 PMOS, U1 INA219, U2 INA219, U3 SunnyBuddy:PRT-12885

Commit message: RTC update
Parts:
- Q3: footprint NMOS:SOT95P230X110-3N -> NMOS:AO3400A
Changed lines of the file:
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@@
 			)
 		)
-		(property "Footprint" "NMOS:SOT95P230X110-3N"
+		(property "Footprint" "NMOS:AO3400A"
 			(at 105.41 106.68 0)
 			(effects

Commit message: Screw matrix update
Parts:
- removed J2: Screw_Terminal_01x02, TerminalBlock_Phoenix:TerminalBlock_Phoenix_MKDS-1,5-2-5.08_1x02_P5.08mm_Horizontal, symbol Connector:Screw_Terminal_01x02
- added J10: Screw_Terminal_01x02, TerminalBlock_Phoenix:TerminalBlock_Phoenix_MKDS-1,5-2_1x02_P5.00mm_Horizontal, symbol Connector:Screw_Terminal_01x02
- J1: footprint TerminalBlock_Phoenix:TerminalBlock_Phoenix_MKDS-1,5-2-5.08_1x02_P5.08mm_Horizontal -> TerminalBlock_Phoenix:TerminalBlock_Phoenix_MKDS-1,5-2_1x02_P5.00mm_Horizontal
Connections:
- net GND: now also J10.2 (Pin_2)
- net Load: now also J10.1 (Pin_1)
