File: Hardware/hw/sensors.kicad_sch (KiCad schematic)
At the start: 10 parts, among them J6 Screw_Terminal_01x04, Q8 NMOS, Q9 NMOS, U11 PESD5V0L2BT,215

Commit message: Sensors update
Parts:
- added J11: Screw_Terminal_01x03, TerminalBlock_Phoenix:TerminalBlock_Phoenix_MKDS-1-3-3.81_1x03_P3.81mm_Horizontal, symbol Connector:Screw_Terminal_01x03
- added J3, J5, J8, J9: Screw_Terminal_01x04, symbol Connector:Screw_Terminal_01x04
- added Q10, Q11, Q12, Q13, Q14, Q15, Q16, Q17: NMOS, symbol Simulation_SPICE:NMOS
- added R36, R37, R42, R43, R48, R49, R54, R55: 4k7, Resistor_SMD:R_0805_2012Metric, symbol Device:R
- added R38, R41, R44, R47, R5, R50, R53, R8: 220, Resistor_SMD:R_0805_2012Metric, symbol Device:R
- added R39, R45, R51, R57, R6: 10k, Resistor_SMD:R_0805_2012Metric, symbol Device:R
- added R40, R46, R52, R7: 100k, Resistor_SMD:R_0805_2012Metric, symbol Device:R
- added R56: 12k, Resistor_SMD:R_0805_2012Metric, symbol Device:R
- added U10, U12, U3, U8: PESD5V0L2BT,215, PESD5V0L2BT,215:SOT95P230X110-3N, symbol PESD5V0L2BT,215:PESD5V0L2BT,215_
- U11: footprint Package_TO_SOT_SMD:SOT-23 -> PESD5V0L2BT,215:SOT95P230X110-3N
Connections:
- net +3V3: now also J11.1 (Pin_1), J3.1 (Pin_1), J5.1 (Pin_1), J8.1 (Pin_1), J9.1 (Pin_1), R36.2, R37.2, R40.2, R42.2, R43.2, R46.2, R48.2, R49.2, R52.2, R54.2, R55.2, R56.2, R7.2
- net GND: now also J11.3 (Pin_3), Q10.3 (S), Q11.3 (S), Q12.3 (S), Q13.3 (S), Q14.3 (S), Q15.3 (S), Q16.3 (S), Q17.3 (S), R39.1, R45.1, R51.1, R57.1, R6.1, U10.3 (GND), U12.3 (GND), U3.3 (GND), U8.3 (GND)
- net GPIO10: now also R38.1, R44.1, R5.1, R50.1
- net I2C_SCL: now also J3.2 (Pin_2), J5.2 (Pin_2), J8.2 (Pin_2), J9.2 (Pin_2), R36.1, R42.1, R48.1, R54.1, U10.1 (IO1), U12.1 (IO1), U3.1 (IO1), U8.1 (IO1)
- net I2C_SDA: now also J3.3 (Pin_3), J5.3 (Pin_3), J8.3 (Pin_3), J9.3 (Pin_3), R37.1, R43.1, R49.1, R55.1, U10.2 (IO2), U12.2 (IO2), U3.2 (IO2), U8.2 (IO2)
- new net: Q12.2 (G), R38.2, R39.2
- new net: Q14.2 (G), R44.2, R45.2
- new net: Q16.1 (D), R52.1, R53.1
- new net: Q16.2 (G), R50.2, R51.2
- new net: Q17.2 (G), R53.2
- new net: Q10.1 (D), R7.1, R8.1
- new net: Q11.2 (G), R8.2
- new net: Q10.2 (G), R5.2, R6.2
- new net: J8.4 (Pin_4), Q15.1 (D)
- new net: Q15.2 (G), R47.2
- new net: Q14.1 (D), R46.1, R47.1
- new net: J5.4 (Pin_4), Q13.1 (D)
- new net: Q13.2 (G), R41.2
- new net: Q12.1 (D), R40.1, R41.1
- new net: J3.4 (Pin_4), Q11.1 (D)
- new net: J9.4 (Pin_4), Q17.1 (D)
- new net ADC3: J11.2 (Pin_2), R56.1, R57.2
Other:
- note added: "2x BH1750"
- note added: "Anemometer"
- note added: "LPS22HB"
- note added: "SHT 40"
- note added: "VEML6075"
- moved on the sheet: J6, Q8, Q9, R30, R31, R32, R33, R34, R35, U11

Commit message: Anemometer update
Parts:
- removed R56: 12k, Resistor_SMD:R_0805_2012Metric, symbol Device:R
- removed R57: 10k, Resistor_SMD:R_0805_2012Metric, symbol Device:R
- added Q18, Q19: NMOS, symbol Simulation_SPICE:NMOS
- added R58, R61: 220, Resistor_SMD:R_0805_2012Metric, symbol Device:R
- added R59: 10k, Resistor_SMD:R_0805_2012Metric, symbol Device:R
- added R60: 100k, Resistor_SMD:R_0805_2012Metric, symbol Device:R
Connections:
- net +3V3: now also R60.2
- net GND: now also Q18.3 (S), Q19.3 (S), R59.1; no longer J11.3 (Pin_3)
- net GPIO10: now also R58.1
- new net: J11.3 (Pin_3), Q19.1 (D)
- new net: Q19.2 (G), R61.2
- new net: Q18.1 (D), R60.1, R61.1
- new net: Q18.2 (G), R58.2, R59.2
Other:
- moved on the sheet: J11, J3, J5, J6, Q10, Q11, Q12, Q13, Q8, Q9, R30, R31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

Commit message: Hardware v1.0
Parts:
- added C13: 100nF, Capacitor_SMD:C_0805_2012Metric, symbol Device:C
- added D2: STS321050B100-EA, Diode_SMD:D_SOD-323, symbol Diode:1N4148WS
- R30: value 220 -> 4k7
- R31: value 100k -> 4k7
- R32: value 10k -> 220
- R33: value 220 -> 10k
- R34: value 4k7 -> 100k
- R35: value 4k7 -> 220
Connections:
- net +3V3: now also R30.2; no longer R35.2
- net ADC3: now also C13.1, D2.2 (A)
- net GND: now also R33.1, C13.2, D2.1 (K); no longer R32.1
- net GPIO10: no longer R30.1, R38.1, R44.1, R50.1, R58.1
- net I2C_SCL: now also R30.1; no longer R34.1
- net I2C_SDA: now also R31.1; no longer R35.1
- net at R7.1, R8.1: now also Q8.1 (D); no longer Q10.1 (D)
- net at Q11.2 (G): now also R35.2; no longer R8.2
- net at R5.2, R6.2: now also Q8.2 (G); no longer Q10.2 (G)
- net at Q9.2 (G): now also R8.2; no longer R33.2
- net at J6.4 (Pin_4): now also Q13.1 (D); no longer Q9.1 (D)
- net at J5.4 (Pin_4): now also Q11.1 (D); no longer Q13.1 (D)
- net at J3.4 (Pin_4): now also Q9.1 (D); no longer Q11.1 (D)
- new net: Q10.1 (D), R34.1, R35.1
- new net: Q10.2 (G), R32.2, R33.2
- new net GPIO11: R32.1
- new net GPIO15: R38.1
- new net GPIO18: R44.1
- new net GPIO19: R50.1
- new net GPIO20: R58.1
Other:
- company: (none) -> UNIZA Faculty of Management Science and Informatics Department of Technical Cybernetics
- title: (none) -> Solar Power Management and Monitoring Circuit
- moved on the sheet: J11, J8, J9, Q14, Q15, Q16, Q17, Q18, Q19, R44, R45, R46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

Commit message: External ADC update
Parts:
- removed R30, R31, R36, R37, R42, R43, R48, R49, R54, R55: 4k7, Resistor_SMD:R_0805_2012Metric, symbol Device:R
- added U13: MCP3422A0-E/SN, MCP3422A7ESN:SOIC127P600X175-8N, symbol MCP3422A7-ESN:MCP3422A0-E/SN
Connections:
- net +3V3: now also U13.3 (Vdd)
- net GND: now also U13.6 (Vss), U13.8 (CH2+)
- net I2C_SCL: now also U13.5 (SCL)
- net I2C_SDA: now also U13.4 (SDA)
- net ADC3 renamed ADC
- net ADC: now also U13.1 (CH1+)
- no-connect marks 0 -> 2
Other:
- moved on the sheet: C13, D2, J11, Q18, Q19, R32, R38, R44, R5, R50, R58, R59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

Commit message: Tomáš update
Parts:
- added C16: 10uF, Capacitor_SMD:C_0805_2012Metric, symbol Device:C
- added C17: 1uF, Capacitor_SMD:C_0805_2012Metric, symbol Device:C
- added C18, C19: 100nF, Capacitor_SMD:C_0805_2012Metric, symbol Device:C
- Q10, Q11, Q12, Q13, Q14, Q15, Q16, Q17, Q18, Q19, Q8, Q9: footprint (none) -> NMOS:SOT95P230X110-3N
- R33, R39, R45, R51, R59, R6: value 10k -> 100k
Connections:
- net +3V3: now also C16.1, C17.1, C18.1, C19.1
- net GND: now also C16.2, C17.2, C18.2, C19.2
Other:
- moved on the sheet: D2, U13

Commit message: little update
Parts:
- removed J11: Screw_Terminal_01x03, TerminalBlock_Phoenix:TerminalBlock_Phoenix_MKDS-1-3-3.81_1x03_P3.81mm_Horizontal, symbol Connector:Screw_Terminal_01x03
- removed J9: Screw_Terminal_01x04, symbol Connector:Screw_Terminal_01x04
- added J10: Screw_Terminal_01x04, TerminalBlock_Phoenix:TerminalBlock_Phoenix_MKDS-1,5-4-5.08_1x04_P5.08mm_Horizontal, symbol Connector:Screw_Terminal_01x04
- added J9: Screw_Terminal_01x03, TerminalBlock_Phoenix:TerminalBlock_Phoenix_MKDS-1,5-3-5.08_1x03_P5.08mm_Horizontal, symbol Connector:Screw_Terminal_01x03
- J3, J5, J6, J8: footprint (none) -> TerminalBlock_Phoenix:TerminalBlock_Phoenix_MKDS-1,5-4-5.08_1x04_P5.08mm_Horizontal
Connections:
- net +3V3: now also J10.1 (Pin_1), J9.1 (Pin_1)
- net ADC: now also J9.2 (Pin_2)
- net I2C_SCL: now also J10.2 (Pin_2)
- net I2C_SDA: now also J10.3 (Pin_3)
- net at Q19.1 (D): now also J9.3 (Pin_3)
- net at Q13.1 (D): now also J5.4 (Pin_4); no longer J6.4 (Pin_4)
- net at Q9.1 (D): now also J10.4 (Pin_4); no longer J3.4 (Pin_4)
- net at Q15.1 (D): now also J6.4 (Pin_4); no longer J8.4 (Pin_4)
- net at Q11.1 (D): now also J3.4 (Pin_4); no longer J5.4 (Pin_4)
- net at Q17.1 (D): now also J8.4 (Pin_4)

Commit message: Mega update
Parts:
- renumbered C19 to C14, C16 to C15, C17 to C16, C18 to C17, C13 to C18, J9 to J10, J10 to J5, J3 to J6, J5 to J7, J6 to J8, J8 to J9, Q12 to Q10, Q9 to Q11, Q11 to Q12, Q16 to Q15, Q15 to Q16, Q10 to Q9, R5 to R21, R32 to R22, R38 to R23, R6 to R24, R33 to R25, R39 to R26, R7 to R27, R34 to R28, R40 to R29, R8 to R30, R35 to R31, R41 to R32, R44 to R33, R50 to R34, R45 to R35, R51 to R36, R46 to R37, R52 to R38, R47 to R39, R53 to R40, R58 to R41, R59 to R42, R60 to R43, R61 to R44, U11 to U10, U10 to U11, U3 to U8, U8 to U9

Commit message: ...
Parts:
- added H1, H2: MountingHole, MountingHole:MountingHole_3.2mm_M3_DIN965_Pad_TopBottom, symbol Mechanical:MountingHole
Changed lines of the file:
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@@
 	)
 	(symbol
+		(lib_id "Mechanical:MountingHole")
+		(at 120.65 154.94 0)
+		(unit 1)
+		(exclude_from_sim no)
+		(in_bom no)
+		(on_board yes)
+		(dnp no)
+		(fields_autoplaced yes)
+		(property "Reference" "H2"
+			(at 123.19 153.6699 0)
+			(effects
+				(font
+					(size 1.27 1.27)
+				)
+				(justify left)
+			)
+		)
+		(property "Value" "MountingHole"
+			(at 123.19 156.2099 0)
+			(effects
+				(font
+					(size 1.27 1.27)
+				)
+				(justify left)
+			)
+		)
+		(property "Footprint" "MountingHole:MountingHole_3.2mm_M3_DIN965_Pad_TopBottom"
+			(at 120.65 154.94 0)
+			(effects
+				(font
+					(size 1.27 1.27)
+				)
+				(hide yes)
+			)
+		)
+		(property "Datasheet" "~"
+			(at 120.65 154.94 0)
+			(effects
+				(font
+					(size 1.27 1.27)
+				)
+				(hide yes)
+			)
+		)
+		(property "Description" "Mounting Hole without connection"
+			(at 120.65 154.94 0)
+			(effects
+				(font
+					(size 1.27 1.27)
+				)
+				(hide yes)
+			)
+		)
+		(instances
+			(project "hw"
+				(path "/e8888c0f-4960-4960-b96f-1ca6e03d7c29/d9cf18c0-974c-45c8-8ea1-a49ffa03ac64"
+					(reference "H2")
+					(unit 1)
+				)
+			)
+		)
+	)
+	(symbol
 		(lib_id "power:+3V3")
 		(at 157.48 29.21 0)
@@
 					(unit 1)
 				)
+			)
+		)
+	)
+	(symbol
+		(lib_id "Mechanical:MountingHole")
+		(at 120.65 144.78 0)
+		(unit 1)
+		(exclude_from_sim no)
+		(in_bom no)
+		(on_board yes)
+		(dnp no)
+		(fields_autoplaced yes)
+		(property "Reference" "H1"
+			(at 123.19 143.5099 0)
+			(effects
+				(font
+					(size 1.27 1.27)
+				)
+				(justify left)
+			)
+		)
+		(property "Value" "MountingHole"
+			(at 123.19 146.0499 0)
+			(effects
+				(font
+					(size 1.27 1.27)
+				)
+				(justify left)
+			)
+		)
+		(property "Footprint" "MountingHole:MountingHole_3.2mm_M3_DIN965_Pad_TopBottom"
+			(at 120.65 144.78 0)
+			(effects
+				(font
+					(size 1.27 1.27)
+				)
+				(hide yes)
+			)
+		)
+		(property "Datasheet" "~"
+			(at 120.65 144.78 0)
+			(effects
+				(font
+					(size 1.27 1.27)
+				)
+				(hide yes)
+			)
+		)
+		(property "Description" "Mounting Hole without connection"
+			(at 120.65 144.78 0)
+			(effects
+				(font
+					(size 1.27 1.27)
+				)
+				(hide yes)
+			)
+		)
+		(instances
+			(project ""
+				(path "/e8888c0f-4960-4960-b96f-1ca6e03d7c29/d9cf18c0-974c-45c8-8ea1-a49ffa03ac64"
+					(reference "H1")
+					(unit 1)
+				)
